File: hardware/plugwatch_G/board/plugwatch.brd (EAGLE design)
At the start: 55.7 x 95.2 mm, 177 parts, among them J1 DM3AT-SF-PEJM5, J2 SCREW_TERMNIAL_1, J3 SCREW_TERMNIAL_1, J4 TC2030-JLINK-L, Q1 NX3008PBK, Q2 MOSFET-NCHANNELSMD, U1 AB1815-T3, U10 STM32L432KC, U11 SIP32510, U12 SIP32510, U13 ADA4096-4ACPZ-R7, U14 SIP32510, U15 REF2030AIDDCR, U16 TCA9406DCUR, U17 SN74LVC1G86DBVR, U18 SN74LVC1G86DBVR, U2 BGA725L6-ALT, U21 SN74LVC1G86DBVR, U22 SN74LVC1G86DBVR, U3 DS2401P+, U4 SAFFB1G56KB0F0A, U5 IRM-03-5V, U6 LIS2DH12, U7 MAX-M8, U8 MAX67XXMAX6749MAX67XX, U9 TPS79330DBVR, X1 ABS07-32.768KHZ-7-T, X2 ABS05-32.768KHZ-T

Commit message: add new plugwatch stuff
Parts:
- removed R45, R48: 1M, passives:0402_RES
- C32, C35: value 10nF -> 1nF
Connections:
- net GND: no longer R45.1, R48.1
- net TDR_L_DETECT: no longer R45.2
- net TDR_N_DETECT: no longer R48.2
Changed lines of the file:
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@@
 <attribute name="VALUE" x="-23.749" y="-305.435" size="1.016" layer="27" font="vector" ratio="12" align="bottom-center"/>
 </element>
-<element name="R45" library="passives" package="0402_RES" value="1M" x="-23.749" y="-307.848" smashed="yes">
-<attribute name="DESCRIPTION" value="RES SMD 100K OHM 1% 1/16W 0402" x="-23.749" y="-307.848" size="1.778" layer="27" display="off"/>
-<attribute name="DIGIKEY" value="541-100KLCT-ND" x="-23.749" y="-307.848" size="1.778" layer="27" display="off"/>
-<attribute name="MANUFACTURER" value="Vishay Dale" x="-23.749" y="-307.848" size="1.778" layer="27" display="off"/>
-<attribute name="MPN" value="CRCW0402100KFKED" x="-23.749" y="-307.848" size="1.778" layer="27" display="off"/>
-<attribute name="NAME" x="-23.749" y="-307.467" size="1.016" layer="25" font="vector" ratio="12" align="bottom-center"/>
-<attribute name="VALUE" x="-23.749" y="-309.245" size="1.016" layer="27" font="vector" ratio="12" align="bottom-center"/>
-</element>
-<element name="C32" library="passives" package="0402_CAP" value="10nF" x="-24.003" y="-311.658" smashed="yes">
+<element name="C32" library="passives" package="0402_CAP" value="1nF" x="-24.003" y="-311.658" smashed="yes">
 <attribute name="DESCRIPTION" value="CAP CER 0.1UF 10V X5R 0402" x="-24.003" y="-311.658" size="1.778" layer="27" display="off"/>
 <attribute name="DIGIKEY" value="311-1336-1-ND" x="-24.003" y="-311.658" size="1.778" layer="27" display="off"/>
@@
 <attribute name="VALUE" x="-24.638" y="-330.708" size="1.016" layer="27" font="vector" ratio="12" align="bottom-center"/>
 </element>
-<element name="R48" library="passives" package="0402_RES" value="1M" x="-17.907" y="-329.311" smashed="yes">
-<attribute name="DESCRIPTION" value="RES SMD 100K OHM 1% 1/16W 0402" x="-23.749" y="-354.076" size="1.778" layer="27" display="off"/>
-<attribute name="DIGIKEY" value="541-100KLCT-ND" x="-23.749" y="-354.076" size="1.778" layer="27" display="off"/>
-<attribute name="MANUFACTURER" value="Vishay Dale" x="-23.749" y="-354.076" size="1.778" layer="27" display="off"/>
-<attribute name="MPN" value="CRCW0402100KFKED" x="-23.749" y="-354.076" size="1.778" layer="27" display="off"/>
-<attribute name="NAME" x="-17.907" y="-328.93" size="1.016" layer="25" font="vector" ratio="12" align="bottom-center"/>
-<attribute name="VALUE" x="-17.907" y="-330.708" size="1.016" layer="27" font="vector" ratio="12" align="bottom-center"/>
-</element>
-<element name="C35" library="passives" package="0402_CAP" value="10nF" x="-19.05" y="-333.121" smashed="yes">
+<element name="C35" library="passives" package="0402_CAP" value="1nF" x="-19.05" y="-333.121" smashed="yes">
 <attribute name="DESCRIPTION" value="CAP CER 0.1UF 10V X5R 0402" x="-24.003" y="-357.886" size="1.778" layer="27" display="off"/>
 <attribute name="DIGIKEY" value="311-1336-1-ND" x="-24.003" y="-357.886" size="1.778" layer="27" display="off"/>
@@
 <contactref element="U22" pad="3"/>
 <contactref element="C31" pad="2"/>
-<contactref element="R45" pad="1"/>
 <contactref element="D25" pad="A"/>
 <contactref element="C32" pad="2"/>
@@
 <contactref element="C33" pad="2"/>
 <contactref element="C34" pad="2"/>
-<contactref element="R48" pad="1"/>
 <contactref element="D28" pad="A"/>
 <contactref element="C35" pad="2"/>
@@
 <wire x1="-24.71293125" y1="-281.94" x2="-23.9776" y2="-274.889" width="0" layer="19" extent="1-1"/>
 <wire x1="-23.56993125" y1="-294.894" x2="-24.71293125" y2="-281.94" width="0" layer="19" extent="1-1"/>
-<wire x1="-24.18206875" y1="-307.848" x2="-23.56993125" y2="-294.894" width="0" layer="19" extent="1-1"/>
-<wire x1="-23.56993125" y1="-311.658" x2="-24.18206875" y2="-307.848" width="0" layer="19" extent="1-1"/>
+<wire x1="-23.56993125" y1="-311.658" x2="-23.56993125" y2="-294.894" width="0" layer="19" extent="1-1"/>
 <wire x1="-23.615" y1="-314.452" x2="-23.56993125" y2="-311.658" width="0" layer="19" extent="1-1"/>
 <wire x1="-23.9776" y1="-324.551" x2="-23.615" y2="-314.452" width="0" layer="19" extent="1-1"/>
 <wire x1="-23.9776" y1="-326.451" x2="-23.9776" y2="-324.551" width="0" layer="19" extent="1-1"/>
 <wire x1="-18.0086" y1="-326.451" x2="-23.9776" y2="-326.451" width="0" layer="19" extent="1-1"/>
-<wire x1="-18.34006875" y1="-329.311" x2="-18.0086" y2="-326.451" width="0" layer="19" extent="1-1"/>
-<wire x1="-18.61693125" y1="-333.121" x2="-18.34006875" y2="-329.311" width="0" layer="19" extent="1-1"/>
+<wire x1="-13.201" y1="-329.057" x2="-18.0086" y2="-326.451" width="0" layer="19" extent="1-1"/>
+<wire x1="-18.61693125" y1="-333.121" x2="-18.0086" y2="-326.451" width="0" layer="19" extent="1-1"/>
 <wire x1="-21.66493125" y1="-333.121" x2="-18.61693125" y2="-333.121" width="0" layer="19" extent="1-1"/>
 <wire x1="-24.71293125" y1="-333.121" x2="-21.66493125" y2="-333.121" width="0" layer="19" extent="1-1"/>
 <wire x1="-22.86" y1="-336.423" x2="-21.66493125" y2="-333.121" width="0" layer="19" extent="1-1"/>
 <wire x1="-21.4122" y1="-336.673" x2="-22.86" y2="-336.423" width="0" layer="19" extent="1-1"/>
-<wire x1="-13.201" y1="-329.057" x2="-18.34006875" y2="-329.311" width="0" layer="19" extent="1-1"/>
 <wire x1="-23.56993125" y1="-189.992" x2="-17.138" y2="-233.553" width="0" layer="19" extent="1-1"/>
 <wire x1="-23.56993125" y1="-187.071" x2="-23.56993125" y2="-189.992" width="0" layer="19" extent="1-1"/>
@@
 <signal name="TDR_L_DETECT">
 <contactref element="D25" pad="C"/>
-<contactref element="R45" pad="2"/>
 <contactref element="R44" pad="1"/>
 <contactref element="C32" pad="1"/>
 <contactref element="U10" pad="10"/>
 <wire x1="-24.18206875" y1="-304.038" x2="-4.425" y2="-101.052" width="0" layer="19" extent="1-1"/>
-<wire x1="-23.31593125" y1="-307.848" x2="-24.18206875" y2="-304.038" width="0" layer="19" extent="1-1"/>
-<wire x1="-24.43606875" y1="-311.658" x2="-23.31593125" y2="-307.848" width="0" layer="19" extent="1-1"/>
+<wire x1="-24.43606875" y1="-311.658" x2="-24.18206875" y2="-304.038" width="0" layer="19" extent="1-1"/>
 <wire x1="-25.915" y1="-314.452" x2="-24.43606875" y2="-311.658" width="0" layer="19" extent="1-1"/>
 </signal>
@@
 <signal name="TDR_N_DETECT">
 <contactref element="D28" pad="C"/>
-<contactref element="R48" pad="2"/>
 <contactref element="R47" pad="1"/>
 <contactref element="C35" pad="1"/>
 <contactref element="U10" pad="11"/>
 <wire x1="-15.501" y1="-329.057" x2="-3.925" y2="-101.052" width="0" layer="19" extent="1-1"/>
-<wire x1="-17.47393125" y1="-329.311" x2="-15.501" y2="-329.057" width="0" layer="19" extent="1-1"/>
-<wire x1="-19.48306875" y1="-333.121" x2="-17.47393125" y2="-329.311" width="0" layer="19" extent="1-1"/>
+<wire x1="-19.48306875" y1="-333.121" x2="-15.501" y2="-329.057" width="0" layer="19" extent="1-1"/>
 <wire x1="-25.07106875" y1="-329.311" x2="-19.48306875" y2="-333.121" width="0" layer="19" extent="1-1"/>
 </signal>

Commit message: add LED with intensity driver to PW, start looking at layout
Parts:
- removed J2, J3: SCREW_TERMNIAL_1, connector:360272-TERMINAL-BLOCK
- removed TP10, TP11, TP12, TP13, TP14, TP15, TP16, TP17, TP18, TP19, TP23, TP24, TP25, TP26, TP27, TP28, TP29, TP30, TP31, TP32, TP4, TP5, TP6, TP7, TP8, TP9: TEST_POINT_0.040IN, headers:TESTPOINT_0.040IN
- added D29: SML-LX0404SIUPGUSB, leds:1MM_SQ_4PAD
- added R45: 1.68k, passives:0402_RES
- added R48: 750, passives:0402_RES
- added R49: 474, passives:0402_RES
- added TP1, TP2: TEST_POINT_0.040IN, headers:TESTPOINT_0.040IN
- added U19: MAX7315ATET, MAX7315ATET:QFN50P300X300X80-17N
Connections:
- removed net AC/L-MEASURE: ASSY1.B5, TP29.TESTPOINT
- removed net AC/L-PERTURB: ASSY1.A0, TP27.TESTPOINT
- removed net AC/L-SENSE: ASSY1.B4, TP31.TESTPOINT
- removed net AC/N-MEASURE: ASSY1.B3, TP28.TESTPOINT
- removed net AC/N-PERTURB: ASSY1.A1, TP32.TESTPOINT
- removed net AC/N-SENSE: ASSY1.B2, TP30.TESTPOINT
- new net N$26: D29.3, R49.1
- new net N$42: D29.4, R48.1
- new net N$49: D29.2, R45.1
- new net N$50: R45.2, U19.2
- new net N$51: R48.2, U19.4
- new net N$52: R49.2, U19.3
- net !EXTERNAL_RST: no longer TP26.TESTPOINT
- net !RTC_CS: no longer TP23.TESTPOINT
- net !RTC_INT1: no longer TP24.TESTPOINT
- net !SD_CS: no longer TP18.TESTPOINT
- net !SD_DETECT: no longer TP11.TESTPOINT
- net ACCEL_INT: no longer TP8.TESTPOINT
- net AC_L_800V_DETECT: now also ASSY1.B5
- net AC_L_LV_OUT: now also ASSY1.A1
- net AC_N: now also TP2.TESTPOINT; no longer J3.P$1, J3.P$2
- net AC_N_800V_DETECT: now also ASSY1.B4
- net AC_N_LV_OUT: now also ASSY1.A0
- net AC_SENSE_PWR_EN: no longer TP10.TESTPOINT
- net GND: now also U19.17, U19.6; no longer TP12.TESTPOINT
- net GPS_PWR_EN: now also ASSY1.C0; no longer ASSY1.D3, TP9.TESTPOINT
- net GPS_RXD: no longer TP6.TESTPOINT
- net GPS_TXD: no longer TP14.TESTPOINT
- net N$12: now also TP1.TESTPOINT; no longer J2.P$1, J2.P$2
- net SD_ENABLE: no longer TP19.TESTPOINT
- net SD_MISO: no longer TP16.TESTPOINT
- net SD_MOSI: no longer TP15.TESTPOINT
- net SD_SCLK: no longer TP17.TESTPOINT
- net SENSORS_SCL: now also U19.12; no longer TP7.TESTPOINT
- net SENSORS_SDA: now also U19.13; no longer TP5.TESTPOINT
- net SERIAL_NUM: no longer TP13.TESTPOINT
- net TDR_L_DETECT: now also ASSY1.B3
- net TDR_L_TRIGGER: now also ASSY1.B1
- net TDR_N_DETECT: now also ASSY1.B2
- net TDR_N_TRIGGER: now also ASSY1.C1
- net VCC: now also D29.1, U19.1, U19.14, U19.15, U19.16; no longer TP4.TESTPOINT
- net WDI: no longer TP25.TESTPOINT
Routing:
- net AC/N-PERTURB: track 97.1 -> 0.00 mm, vias 1 -> 0
- net AC/N-SENSE: track 92.2 -> 0.00 mm, vias 1 -> 0
- net AC/N-MEASURE: track 85.2 -> 0.00 mm, vias 1 -> 0
- net AC/L-PERTURB: track 84.5 -> 0.00 mm, vias 1 -> 0
- net AC_L_LV_OUT: track 0.00 -> 84.0 mm, vias 0 -> 1
- net TDR_N_DETECT: track 0.00 -> 82.5 mm, vias 0 -> 1
- net AC/L-MEASURE: track 80.3 -> 0.00 mm, vias 1 -> 0
- net TDR_L_DETECT: track 0.00 -> 78.0 mm, vias 0 -> 1
- net AC/L-SENSE: track 77.7 -> 0.00 mm, vias 1 -> 0
- net AC_N_LV_OUT: track 0.00 -> 76.8 mm, vias 0 -> 1
- net AC_L_800V_DETECT: track 0.00 -> 72.3 mm, vias 0 -> 1
- net GPS_PWR_EN: track 60.9 -> 19.5 mm
- net SENSORS_SCL: track 42.0 -> 10.1 mm, vias 1 -> 0
- net VCC: track 186.3 -> 155.9 mm
- net AC_N: track 30.8 -> 4.48 mm, vias 1 -> 0
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Other:
- board text removed: "!ExRST"
- board text removed: "!RTCS"
- board text removed: "!RTINT"
- board text removed: "!SDCS"
- board text removed: "!SDDET"
- board text removed: "3V3"
- board text removed: "AC/L/M"
- board text removed: "AC/L/P"
- board text removed: "AC/L/S"
- board text removed: "AC/N/M"
- board text removed: "AC/N/S"
- board text removed: "ACEN"
- board text removed: "GND"
- board text removed: "GRX"
- board text removed: "GTX"
- board text removed: "INT"
- board text removed: "MISO"
- board text removed: "MOSI"
- board text removed: "SCL"
- board text removed: "SCLK"
- board text removed: "SDA"
- board text removed: "SDEN"
- board text removed: "SN"
- board text removed: "WDI"
- board text removed: "WiRX"

Commit message: make significant layout progress
Parts:
- removed U$3: (no value), logos:UCB_CAL_200MIL
- added C36: 0.1uF, passives:0402_CAP
- added C37: 1uF, passives:0402_CAP
- U17, U18, U21, U22: value SN74LVC1G86DBVR -> SN74LVC1G86DRLRDRL5-L; device SN74LVC:DBV5 -> SN74LVC1G86:DRL5-L
- moved TP1 369.7 mm to (38.7, 27.6)
- moved C35 369.3 mm to (4.45, 35.4), turned to 270 degrees
- moved C34 369.1 mm to (5.71, 34.9), turned to 180 degrees
- moved C33 368.8 mm to (3.17, 34.5), turned to 180 degrees
- moved TP2 367.7 mm to (15.5, 27.8)
- moved R47 366.5 mm to (5.71, 35.9)
- moved U13 365.9 mm to (5.21, 28.4)
- moved D28 365.1 mm to (2.16, 35.7), turned to 180 degrees
- moved R46 363.3 mm to (3.68, 33.1), turned to 270 degrees
- moved U17 359.4 mm to (2.03, 33.0)
- moved U18 359.2 mm to (5.33, 33.0)
- moved D25 356.6 mm to (2.29, 41.1), turned to 180 degrees
- moved D27 355.7 mm to (9.78, 35.6)
- moved D26 353.9 mm to (9.91, 33.1), turned to 180 degrees
- moved C32 353.6 mm to (4.70, 40.8), turned to 270 degrees
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Connections:
- new net BOOT0: R37.2, U10.31
- net !RST: no longer R37.2, U10.31
- net AC_COPROC_VCC: now also C36.1, C37.1
- net GND: now also C36.2, C37.2
Routing:
- net TDR_N_DETECT: track 82.5 -> 9.84 mm, vias 1 -> 0
- net TDR_L_DETECT: track 78.0 -> 12.1 mm, vias 1 -> 0
- net AC_L_LV_OUT: track 84.0 -> 21.6 mm, vias 1 -> 0
- net AC_N_LV_OUT: track 76.8 -> 19.2 mm, vias 1 -> 0
- net AC_L_800V_DETECT: track 72.3 -> 16.8 mm, vias 1 -> 0
- net GPS_RXD: track 41.9 -> 1.90 mm, vias 1 -> 0
- net VCC: track 155.9 -> 119.5 mm, vias 9 -> 8
- net AC_SENSE_PWR_EN: track 63.4 -> 30.4 mm, vias 1 -> 0
- net GPS_TXD: track 42.8 -> 21.4 mm, vias 1 -> 0
- net VCC_RF: track 17.8 -> 2.09 mm
- net 5V: track 178.5 -> 165.9 mm, vias 5 -> 4
- net GPS_PWR_EN: track 19.5 -> 7.01 mm
- net GPS_RF_IN: track 7.09 -> 0.00 mm
- net !EXTERNAL_RST: track 34.3 -> 40.1 mm
- net N$23: track 33.9 -> 28.7 mm
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- removed copper zone on layer 1, net GPS_VCC
- removed copper zone on layer 1, net N$7
- removed copper zone on layer 15, net N$7
- removed copper zone on layer 16, net N$7
- removed copper zone on layer 2, net N$7
Other:
- board text removed: "NEUTRAL"
