File: hardware/plugwatch_G/board/plugwatch.brd (EAGLE design)
At the start: 55.7 x 95.2 mm, 155 parts, among them J1 DM3AT-SF-PEJM5, J4 TC2030-JLINK-L, Q1 NX3008PBK, Q2 MOSFET-NCHANNELSMD, U1 AB1815-T3, U10 STM32L432KC, U11 SIP32510, U12 SIP32510, U13 ADA4096-4ACPZ-R7, U14 SIP32510, U15 REF2030AIDDCR, U16 TCA9406DCUR, U17 SN74LVC1G86DRLRDRL5-L, U18 SN74LVC1G86DRLRDRL5-L, U19 MAX7315ATET, U2 BGA725L6-ALT, U21 SN74LVC1G86DRLRDRL5-L, U22 SN74LVC1G86DRLRDRL5-L, U3 DS2401P+, U4 SAFFB1G56KB0F0A, U5 IRM-03-5V, U6 LIS2DH12, U7 MAX-M8, U8 MAX67XXMAX6749MAX67XX, U9 TPS79330DBVR, X1 ABS07-32.768KHZ-7-T, X2 ABS05-32.768KHZ-T

Commit message: finish routing board
Parts:
- removed C27, C29: 0.01uF, passives:0402_CAP
- removed D11, D20: 3V, SparkFun-DiscreteSemi:SOD-323
- removed D12, D13, D14, D3, D4, D5: 200V, diode:DO214AA
- removed D2, D22: 2000Vr, diode:DO214AC
- removed R39, R42: 10, passives:0402_RES
- moved D19 28.4 mm to (7.11, 8.89), flipped to the bottom, turned to 0 degrees
- moved C28 25.1 mm to (7.75, 10.4), flipped to the bottom, turned to 0 degrees
- moved D15 25.0 mm to (12.7, 8.89), flipped to the bottom
- moved C26 20.7 mm to (7.49, 17.4), flipped to the bottom
- moved D10 20.2 mm to (6.86, 15.5), flipped to the bottom
- moved D1 18.9 mm to (44.5, 16.0), flipped to the bottom
- moved D16 17.6 mm to (20.1, 8.89), flipped to the bottom
- moved U14 17.1 mm to (19.6, 48.8), turned to 270 degrees
- moved R26 16.3 mm to (19.6, 46.5), turned to 180 degrees
- moved D6 14.6 mm to (12.7, 16.0), flipped to the bottom
- moved R38 13.9 mm to (39.9, 16.0), flipped to the bottom
- moved U15 11.8 mm to (19.3, 43.4), turned to 180 degrees
- moved C23 11.0 mm to (4.83, 54.6), turned to 180 degrees
- moved U9 10.4 mm to (19.3, 53.3), turned to 90 degrees
- moved R6 10.4 mm to (10.2, 34.3), turned to 180 degrees
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Connections:
- net GND1 renamed A
- net GND2 renamed A2
- removed net AC_L_600V_DETECT: C27.1, D11.C, D4.A, U10.28
- removed net AC_N_600V_DETECT: C29.1, D13.A, D20.C, U10.30
- removed net N$1: D3.C, D5.A
- removed net N$22: D5.C, R39.1
- removed net N$24: D3.A, D4.C
- removed net N$33: D2.C, R39.2
- removed net N$34: D12.C, D14.A
- removed net N$43: D12.A, D13.C
- removed net N$45: D14.C, R42.1
- removed net N$48: D22.C, R42.2
- net AC_L_800V_DETECT: now also ASSY1.B1; no longer ASSY1.B5
- net AC_L_HV_OUT: now also U10.6; no longer U10.8
- net AC_L_LV_OUT: now also U10.9; no longer U10.6
- net AC_L_SENSE: no longer D2.A
- net AC_N: no longer D22.A
- net AC_N_800V_DETECT: now also ASSY1.C1; no longer ASSY1.B4
- net AC_N_HV_OUT: now also U10.8; no longer U10.9
- net GND: no longer C27.2, C29.2, D11.A, D20.A
- net TDR_L_DETECT: now also ASSY1.B2, U10.13; no longer ASSY1.B3, U10.10
- net TDR_L_TRIGGER: now also ASSY1.B3; no longer ASSY1.B1
- net TDR_N_DETECT: now also ASSY1.B4; no longer ASSY1.B2
- net TDR_N_TRIGGER: now also ASSY1.B5, U10.10; no longer ASSY1.C1, U10.13
Routing:
- net AC_COPROC_VCC: track 0.00 -> 99.4 mm, vias 0 -> 2
- net TDR_N_TRIGGER: track 0.00 -> 88.7 mm, vias 0 -> 2
- net !RST: track 0.00 -> 84.9 mm, vias 0 -> 2
- net VCC: track 119.5 -> 197.7 mm, vias 8 -> 9
- net AC_L_800V_DETECT: track 16.8 -> 92.1 mm, vias 0 -> 1
- net TDR_N_DETECT: track 9.84 -> 84.1 mm, vias 0 -> 2
- net SWDIO: track 0.00 -> 73.9 mm, vias 0 -> 2
- net SWDCLK: track 0.00 -> 72.7 mm, vias 0 -> 2
- net AC_N_800V_DETECT: track 0.00 -> 72.0 mm, vias 0 -> 1
- net AC_L_LV_OUT: track 21.6 -> 90.3 mm, vias 0 -> 2
- net TDR_L_TRIGGER: track 0.00 -> 67.5 mm, vias 0 -> 2
- net AC_N_LV_OUT: track 19.2 -> 83.9 mm, vias 0 -> 2
- net AC_SENSE_VCC: track 0.95 -> 65.0 mm, vias 0 -> 6
- net AC_N: track 0.00 -> 54.5 mm, vias 0 -> 2
- net !RTC_INT2: track 0.00 -> 53.5 mm, vias 0 -> 3
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- added copper zone on layer 1, net AC_L_SENSE
- added copper zone on layer 1, net AC_N
- added copper zone on layer 1, net GPS_VCC
Other:
- board text removed: "HIGH VOLTAGE"
- board text removed: "LINE"

Commit message: fix up names and board documentation
Parts:
- moved C7 5.80 mm to (45.5, 64.3)
- moved R4 1.52 mm to (44.1, 26.3)
- moved C3 1.02 mm to (43.2, 58.9)
- moved U21 0.51 mm to (3.94, 38.9)
- moved U17 0.51 mm to (3.30, 24.1)
- moved TP1 0.40 mm to (36.6, 26.4)
- moved R46 0.25 mm to (5.21, 24.3)
- moved U18 0.25 mm to (7.37, 24.1)
- moved U22 0.25 mm to (7.87, 38.9)
- moved C14 0.25 mm to (43.2, 57.1)
Routing:
- net N$2: track 24.6 -> 27.0 mm
- net AC_SENSE_VCC: track 65.0 -> 63.9 mm
- net !RST1: track 2.29 -> 3.05 mm
- net !RST2: track 2.42 -> 3.18 mm
- net GND: vias 75 -> 76
Other:
- board text added: "nLine, Inc."

Commit message: renumber components, add cutout
Parts:
- removed C36: 0.1uF, passives:0402_CAP
- removed R48: 750, passives:0402_RES
- removed R49: 474, passives:0402_RES
- removed U22: SN74LVC1G86DRLRDRL5-L, SN74LVC1G86:DRL5-L
- added C29: 4.7uF, passives:0402_CAP
- added R39, R42: 953k, passives:0402_RES
- added U20: TCA9406DCUR, tca9406:DCU8
- C1: value 47pF -> 4.3pF
- C10: value 1uF -> 10nF
- C11: value 0.1uF -> 10nF
- C12: value 4.7uF -> 10nF
- C13: value 10uF -> 10nF
- C14: value 10uF -> 0.1uF
- C15, C16: value 100uF -> 0.1uF; device passives:1210_CAP -> passives:0402_CAP
- C17: value 2000uF -> 0.1uF; device rcl:E5-13 -> passives:0402_CAP
- C2: value 10nF -> 4.3pF
- C20, C22: value 1uF -> 0.1uF
- C23: value 4.7uF -> 0.82uF
- C24, C25: value 4.3pF -> 1uF
- C26: value 0.01uF -> 1uF
- C28: value 0.01uF -> 2.2uF
- C3: value 10nF -> 47pF
- C30: value 100pF -> 4.7uF
- C31: value 10nF -> 10uF
- C32: value 1nF -> 10uF
- C33: value 100pF -> 100uF; device passives:0402_CAP -> passives:1210_CAP
- C34: value 10nF -> 100uF; device passives:0402_CAP -> passives:1210_CAP
- C35: value 1nF -> 2000uF; device passives:0402_CAP -> rcl:E5-13
- C4, C5: value 0.1uF -> 100pF
- C6, C7: value 0.1uF -> 1nF
- C8: value 2.2uF -> 10nF
- C9: value 0.82uF -> 10nF
- L1: value 5.6nH -> 5.6n
- Q1: value NX3008PBK -> MOSFET-NCHANNELSMD
- Q2: value MOSFET-NCHANNELSMD -> NX3008PBK
- R1: value 66.5K -> 1; device passives:0402_RES -> resistor:R2512
- R10: value 10k -> 1.68k
- R11, R12: value 10k -> 3.74k
- R13: value 10k -> 5.1k
- R19: value 34k -> 10k
- R2: value 100k -> 10
- R20, R21, R22, R24: value 100k -> 10k
- R23: value 953k -> 10k
- R25: value 100k -> 34k
- R26: value 100k -> 66.5k
- R27: value 1M -> 100k
- R28, R30, R31: value 953k -> 100k
- R29: value 3.74k -> 100k
- R3: value 1M -> 10
- R32: value 825k -> 100k
- R33: value 1.00k -> 100k
- R34, R35: value 953k -> 800k
- R36: value 1.00k -> 825k
- R37: value 10k -> 953k
- R38, R40: value 10 -> 953k
- R4: value 1 -> 40; device resistor:R2512 -> passives:0402_RES
- R41: value 1M -> 953k
- R43: value 40 -> 953k
- R44: value 800k -> 953k
- R45: value 1.68k -> 1M
- R46: value 40 -> 1M
- R47: value 800k -> 1M
- R5: value 3.74k -> 40
- R6: value 953k -> 474
- R7: value 953k -> 750
- R8: value 5.1k -> 1.00k
- R9: value 10k -> 1.00k
- U10: value STM32L432KC -> MAX7315ATET; device chips:UQFN-32 -> MAX7315ATET:QFN50P300X300X80-17N
- U11: value SIP32510 -> REF2030AIDDCR; device chips:TSOT23-6 -> ref2033:DDC5
- U13: value ADA4096-4ACPZ-R7 -> SIP32510; device ada4096-4:CP_16_27 -> chips:TSOT23-6
- U15: value REF2030AIDDCR -> SN74LVC1G86DRLRDRL5-L; device ref2033:DDC5 -> SN74LVC1G86:DRL5-L
- U16: value TCA9406DCUR -> SN74LVC1G86DRLRDRL5-L; device tca9406:DCU8 -> SN74LVC1G86:DRL5-L
- U19: value MAX7315ATET -> STM32L432KC; device MAX7315ATET:QFN50P300X300X80-17N -> chips:UQFN-32
- U2: value BGA725L6-ALT -> ADA4096-4ACPZ-R7; device Particle:LNA-TSLP-6-2-ALT -> ada4096-4:CP_16_27
- U21: value SN74LVC1G86DRLRDRL5-L -> TPS79330DBVR; device SN74LVC1G86:DRL5-L -> tps7933:DBV5
- U3: value DS2401P+ -> BGA725L6-ALT; device DS2401P+:21-0382 -> Particle:LNA-TSLP-6-2-ALT
- U4: value SAFFB1G56KB0F0A -> DS2401P+; device Particle:QCS5I -> DS2401P+:21-0382
- U5: value IRM-03-5V -> SAFFB1G56KB0F0A; device powerwatch:IRM-03 -> Particle:QCS5I
- U6: value LIS2DH12 -> IRM-03-5V; device chips:LGA-12 -> powerwatch:IRM-03
- U7: value MAX-M8 -> LIS2DH12; device u-blox:MAX-M8 -> chips:LGA-12
- U8: value MAX67XXMAX6749MAX67XX -> MAX-M8; device chips:SOT-23-8 -> u-blox:MAX-M8
- U9: value TPS79330DBVR -> MAX67XXMAX6749MAX67XX; device tps7933:DBV5 -> chips:SOT-23-8
- X1: value ABS07-32.768KHZ-7-T -> ABS05-32.768KHZ-T; device crystals:2-SMD -> crystals:ABS05
- X2: value ABS05-32.768KHZ-T -> ABS07-32.768KHZ-7-T; device crystals:ABS05 -> crystals:2-SMD
- moved R2 73.1 mm to (39.9, 16.0), flipped to the bottom, turned to 180 degrees
- moved C15 69.9 mm to (20.3, 77.2), turned to 0 degrees
- moved R33 69.3 mm to (43.3, 89.0)
- moved U6 63.2 mm to (27.9, 12.7), turned to 0 degrees
- moved R1 60.9 mm to (44.1, 26.3), flipped to the bottom
- moved C28 57.7 mm to (31.0, 63.2), flipped to the top, turned to 90 degrees
- moved C10 57.4 mm to (7.49, 17.4), flipped to the bottom, turned to 0 degrees
- moved R6 56.7 mm to (16.3, 90.7), turned to 0 degrees
- moved R7 55.0 mm to (16.3, 89.3)
- moved C7 54.4 mm to (6.10, 26.7), turned to 270 degrees
- moved R28 53.5 mm to (27.7, 77.5), turned to 0 degrees
- moved U4 52.5 mm to (3.05, 80.5), turned to 270 degrees
- moved R3 52.2 mm to (39.9, 8.89), flipped to the bottom, turned to 180 degrees
- moved R29 51.8 mm to (42.7, 63.5), turned to 0 degrees
- moved U3 51.8 mm to (44.7, 49.8), turned to 180 degrees
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- renumbered C37 to C27, J4 to J2
Connections:
- net !EXTERNAL_RST: now also R22.2, U9.7; no longer R17.2, U8.7
- net !RST: now also U19.4; no longer U10.4
- net !RST1: now also R4.2, U15.4, U16.2; no longer R43.2, U21.4, U22.2
- net !RST2: now also R5.2; no longer R46.2
- net !RTC_CS: now also R21.2, R23.2; no longer R16.2, R18.2
- net !RTC_INT1: now also R20.2; no longer R15.2
- net !RTC_INT2: now also Q2.1, R33.2; no longer Q1.1, R2.2
- net !SD_CS: now also R16.1; no longer R11.1
- net !SD_DETECT: now also R27.1; no longer R20.1
- net 5V: now also C33.1, C34.1, C35.+, R25.1, R30.1, R46.1, U6.V+; no longer C15.1, C16.1, C17.+, R19.1, R24.1, R41.1, U5.V+
- net A: now also C4.1, R4.1, U16.1; no longer C30.1, R43.1, U22.1
- net A2: now also C5.1, R5.1; no longer C33.1, R46.1
- net ACCEL_INT: now also U7.12; no longer U6.12
- net AC_COPROC_VCC: now also C26.1, C30.1, U19.1, U19.17, U20.3, U20.6, U21.5; no longer C23.1, C36.1, U10.1, U10.17, U16.3, U16.6, U9.5
- net AC_L_800V_DETECT: now also C10.1, U19.27; no longer C26.1, U10.27
- net AC_L_HV_OUT: now also R8.2, U19.6, U2.14; no longer R33.2, U10.6, U13.14
- net AC_L_LV_OUT: now also R11.2, U19.9, U2.7; no longer R5.2, U10.9, U13.7
- net AC_L_SENSE: now also R1.1, R37.1, R42.2; no longer R31.2, R4.1, R6.1
- net AC_N: now also R39.1, R43.2, U6.AC/N; no longer R23.1, R34.2, U5.AC/N
- net AC_N1: now also U16.4; no longer U22.4
- net AC_N_800V_DETECT: now also C11.1, U19.29; no longer C28.1, U10.29
- net AC_N_HV_OUT: now also R9.2, U19.8, U2.6; no longer R36.2, U10.8, U13.6
- net AC_N_LV_OUT: now also R12.1, U19.7, U2.15; no longer R29.1, U10.7, U13.15
- net AC_SCL: now also U19.19, U20.5; no longer U10.19, U16.5
- net AC_SDA: now also U19.20, U20.4; no longer U10.20, U16.4
- net AC_SENSE_PWR_EN: now also R32.2; no longer R26.2
- net AC_SENSE_VCC: now also U11.3, U11.4, U15.5, U16.5, U21.1, U21.3; no longer U15.3, U15.4, U21.5, U22.5, U9.1, U9.3
- net BOOT0: now also R24.2, U19.31; no longer R37.2, U10.31
- net GND: now also C1.1, C17.2, C24.2, C25.2, C29.2, C3.2, C32.1, C35.-, C7.2, C8.1, C9.1, Q1.2, R19.2, R24.1, R26.2, R29.1, R31.2, R32.1, R38.1, R40.1, R41.2, R44.2, R45.2, R47.2, U10.17, U10.6, U11.2, U13.4, U15.1, U15.3, U16.3, U19.16, U19.32, U19.THERMAL, U2.10, U2.17, U20.2, U21.2, U3.4, U4.1, U5.2, U5.3, U5.5, U6.V-, U7.3, U7.5, U7.6, U7.7, U7.8, U8.1, U8.10, U8.12, U9.4; no longer C1.2, C17.-, C24.1, C25.1, C3.1, C32.2, C35.2, C36.2, C7.1, C8.2, C9.2, Q2.2, R1.2, R14.2, R21.1, R22.1, R25.2, R26.1, R27.2, R3.2, R30.2, R35.2, R37.1, R7.1, U10.16, U10.32, U10.THERMAL, U11.4, U13.10, U13.17, U15.2, U16.2, U19.17, U19.6, U2.1, U2.4, U21.1, U21.3, U22.3, U4.2, U4.3, U4.5, U5.V-, U6.3, U6.5, U6.6, U6.7, U6.8, U7.1, U7.10, U7.12, U8.4, U9.2
- net GPS_PPS: now also U19.26, U8.4; no longer U10.26, U7.4
- net GPS_PWR_EN: now also R29.2, U12.3; no longer R22.2, U11.3
- net GPS_RF_IN: now also U5.4, U8.11; no longer U4.4, U7.11
- net GPS_VCC: now also C32.2, C9.2, U12.1, U12.2, U8.6, U8.7, U8.8; no longer C3.2, C7.2, U11.1, U11.2, U7.6, U7.7, U7.8
- net LNA_IN: now also U3.5; no longer U2.5
- net LNA_OUT: now also U3.3, U5.1; no longer U2.3, U4.1
- net N$10: now also Q2.3, R25.2, R26.1; no longer Q1.3, R1.1, R19.2
- net N$11: now also C1.2, U19.2, X1.B; no longer C24.2, U10.2, X2.B
- net N$13: now also C3.1; no longer C1.1
- net N$17: now also C13.1, R35.2; no longer C34.1, R47.2
- net N$18: now also C29.1, R15.2, R16.2, R17.2, R27.2, U13.1, U13.2; no longer C12.1, R10.2, R11.2, R12.2, R20.2, U12.1, U12.2
- net N$2: now also R1.2, U6.AC/L; no longer R4.2, U5.AC/L
- net N$20: now also X2.2; no longer X1.2
- net N$21: now also X2.1; no longer X1.1
- net N$23: now also R22.1, R36.1, U9.5, U9.8; no longer R17.1, R32.1, U8.5, U8.8
- net N$25: now also R30.2, R31.1; no longer R24.2, R25.1
- net N$26: now also R6.1; no longer R49.1
- net N$3: now also R12.2, R39.2, R40.2, U2.1; no longer R23.2, R28.2, R29.2, U13.1
- net N$30: now also R2.1; no longer R38.1
- net N$31: now also Q1.3, R36.2, R45.1, R46.2, U9.1; no longer Q2.3, R27.1, R32.2, R41.2, U8.1
- net N$32: now also R2.2; no longer R38.2
- net N$36: now also C23.1, U9.3; no longer C9.1, U8.3
- net N$39: now also C28.1, U9.2; no longer C8.1, U8.2
- net N$4: now also R11.1, R37.2, R38.2, U2.8; no longer R5.1, R6.2, R7.2, U13.8
- net N$40: now also U8.2; no longer U7.2
- net N$41: now also U8.3; no longer U7.3
- net N$42: now also R7.1; no longer R48.1
- net N$44: now also C12.1, R34.2; no longer C31.1, R44.2
- net N$46: now also R3.1; no longer R40.1
- net N$47: now also R3.2; no longer R40.2
- net N$49: now also R10.1; no longer R45.1
- net N$5: now also R23.1; no longer R18.1
- net N$50: now also R10.2, U10.2; no longer R45.2, U19.2
- net N$51: now also R7.2, U10.4; no longer R48.2, U19.4
- net N$52: now also R6.2, U10.3; no longer R49.2, U19.3
- net N$6: now also R41.1, R42.1, R8.1, U2.12; no longer R30.1, R31.1, R33.1, U13.12
- net N$8: now also R43.1, R44.1, R9.1, U2.5; no longer R34.1, R35.1, R36.1, U13.5
- net N$9: now also C2.2, U19.3, X1.A; no longer C25.2, U10.3, X2.A
- net PARTICLE_RST: now also Q1.1, R47.1; no longer Q2.1, R3.1
- net REF_1V5: now also C16.1, C17.1, C19.1, U11.1, U2.11, U2.2, U2.4, U2.9; no longer C11.1, C5.1, C6.1, U13.11, U13.2, U13.4, U13.9, U15.1
- net REF_3V: now also C25.1, U11.5, U19.5, U2.3; no longer C19.1, U10.5, U13.3, U15.5
- net SD_ENABLE: now also R28.2, U13.3; no longer R21.2, U12.3
- net SD_MISO: now also R17.1; no longer R12.1
- net SD_MOSI: now also R15.1; no longer R10.1
- net SENSORS_SCL: now also R18.1, U10.12, U20.8, U7.1; no longer R13.1, U16.8, U19.12, U6.1
- net SENSORS_SDA: now also R14.1, U10.13, U20.1, U7.4; no longer R9.1, U16.1, U19.13, U6.4
- net SERIAL_NUM: now also R13.2, U4.2; no longer R8.2, U3.2
- net SWDCLK: now also U19.24; no longer U10.24
- net SWDIO: now also U19.23; no longer U10.23
- net TDR_L_DETECT: now also C6.1, R34.1, U19.13; no longer C32.1, R44.1, U10.13
- net TDR_L_TRIGGER: now also U15.2, U19.12; no longer U10.12, U21.2
- net TDR_N_DETECT: now also C7.1, R35.1, U19.11; no longer C35.1, R47.1, U10.11
- net TDR_N_TRIGGER: now also U19.10; no longer U10.10
- net VCC: now also C15.1, C24.1, C31.1, Q2.2, R13.1, R14.2, R18.2, R20.1, R21.1, R33.1, U10.1, U10.14, U10.15, U10.16, U13.5, U13.6, U20.7, U7.10, U7.2, U7.9; no longer C10.1, C13.1, C4.1, Q1.2, R13.2, R15.1, R16.1, R2.1, R8.1, R9.2, U11.5, U11.6, U16.7, U19.1, U19.14, U19.15, U19.16, U6.10, U6.2, U6.9
- net VCC_RF: now also C8.2, U3.2, U3.6, U8.14; no longer C2.2, U2.2, U2.6, U7.14
- net WDI: now also R19.1, U9.6; no longer R14.1, U8.6
Routing:
- net AC_N: track 54.5 -> 60.2 mm
- net AC_L_SENSE: track 51.0 -> 54.2 mm
- net GND: vias 76 -> 78
- added copper zone on layer 1, net NOTHING
- added copper zone on layer 15, net NOTHING
- added copper zone on layer 16, net NOTHING
- added copper zone on layer 2, net NOTHING
- removed copper zone on layer 1, net AC_L_SENSE
- removed copper zone on layer 1, net AC_N

Commit message: add board and schematic with final part numbers
Parts:
- removed D21, D23, D26: 2000Vr, diode:DO214AC
- removed D24, D27: >1kVr, diode:DO214AC
- removed D25, D28: 3V, SparkFun-DiscreteSemi:SOD-323
- added D11, D12, D13: 200V, diode:DO214AA
- added D14: 1000Vr, diode:DO214AC
- added D2, D3, D4: 3V, SparkFun-DiscreteSemi:SOD-323
- added D5: LED0603, leds:LED-0603
- added R48: 1M, passives:0402_RES
- C12, C13: device passives:0402_CAP -> SparkFun-Capacitors:1206
- D1: value 2000Vr -> 3V; device diode:DO214AC -> SparkFun-DiscreteSemi:SOD-323
- D10: value 3V -> 200V; device SparkFun-DiscreteSemi:SOD-323 -> diode:DO214AA
- D15, D16, D17, D18: value 200V -> 1000Vr; device diode:DO214AA -> diode:DO214AC
- D19: value 3V -> 1000Vr; device SparkFun-DiscreteSemi:SOD-323 -> diode:DO214AC
- R10: value 1.68k -> 1.69k
- R11: value 3.74k -> 1.69k
- R13: value 5.1k -> 3.74k
- R14: value 10k -> 5.1k
- R25: value 34k -> 10k
- R26: value 66.5k -> 34k
- R27: value 100k -> 66.5k
- R34: value 800k -> 100k
- R35: value 800k -> 806k; device passives:0402_RES -> passives:0805_RES
- R36: value 825k -> 806k; device passives:0402_RES -> passives:0805_RES
- R37: value 953k -> 825k
- R38, R39, R40, R41, R42, R43, R44: device passives:0402_RES -> passives:0805_RES
- R4, R5: value 40 -> 40.2
- R45: value 1M -> 953k; device passives:0402_RES -> passives:0805_RES
- R6: value 474 -> 475
- moved R34 59.0 mm to (43.3, 89.0), turned to 270 degrees
- moved R13 52.6 mm to (1.52, 32.0), turned to 270 degrees
- moved R33 48.7 mm to (19.6, 46.5), turned to 180 degrees
- moved R25 44.7 mm to (7.11, 53.8), turned to 180 degrees
- moved R45 38.0 mm to (6.86, 30.1), turned to 180 degrees
- moved D1 37.6 mm to (6.86, 15.5), turned to 0 degrees
- moved R36 37.5 mm to (8.89, 27.9)
- moved R30 37.5 mm to (42.7, 63.5), turned to 0 degrees
- moved D17 31.9 mm to (13.0, 37.3), flipped to the top, turned to 270 degrees
- moved D15 31.8 mm to (44.5, 8.89), turned to 180 degrees
- moved R37 31.4 mm to (27.2, 60.7), turned to 0 degrees
- moved R32 31.2 mm to (7.37, 75.2), turned to 0 degrees
- moved D16 28.9 mm to (15.2, 37.3), flipped to the top, turned to 90 degrees
- moved D18 28.2 mm to (14.7, 28.7), flipped to the top, turned to 270 degrees
- moved R22 25.0 mm to (3.94, 76.2), turned to 180 degrees
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Connections:
- new net N$1: D5.C, R11.2
- new net N$7: D5.A, U19.15
- net !EXTERNAL_RST: now also R23.2; no longer R22.2
- net !RTC_CS: now also R22.2, R24.2; no longer R21.2, R23.2
- net !RTC_INT1: now also R21.2; no longer R20.2
- net !RTC_INT2: now also R34.2; no longer R33.2
- net !SD_CS: now also R17.1; no longer R16.1
- net !SD_DETECT: now also R28.1; no longer R27.1
- net 5V: now also R26.1, R31.1, R47.1; no longer R25.1, R30.1, R46.1
- net AC_L_800V_DETECT: now also D1.C; no longer D10.C
- net AC_L_LV_OUT: now also R12.2; no longer R11.2
- net AC_L_SENSE: now also D14.A, D16.C, D17.A, R38.1, R43.2; no longer D1.A, D23.C, D24.A, R37.1, R42.2
- net AC_N: now also D15.A, D18.C, D19.A, R40.1, R44.2; no longer D21.A, D26.C, D27.A, R39.1, R43.2
- net AC_N1: now also D16.A; no longer D23.A
- net AC_N2: now also D18.A; no longer D26.A
- net AC_N_800V_DETECT: now also D10.A, D2.C; no longer D15.A, D19.C
- net AC_N_LV_OUT: now also R13.1; no longer R12.1
- net AC_SENSE_PWR_EN: now also R33.2; no longer R32.2
- net BOOT0: now also R25.2; no longer R24.2
- net GND: now also D1.A, D2.A, D3.A, D4.A, R11.1, R20.2, R25.1, R27.2, R30.1, R32.2, R33.1, R39.1, R41.1, R42.2, R46.2, R48.2; no longer D10.A, D19.A, D25.A, D28.A, R19.2, R24.1, R26.2, R28.1, R31.2, R32.1, R38.1, R40.1, R41.2, R44.2, R47.2
- net GPS_PWR_EN: now also R30.2; no longer R29.2
- net N$10: now also R26.2, R27.1; no longer R25.2, R26.1
- net N$17: now also D19.C, R36.2; no longer D27.C, R35.2
- net N$18: now also R18.2, R28.2; no longer R15.2, R27.2
- net N$23: now also R23.1, R37.1; no longer R22.1, R36.1
- net N$25: now also R31.2, R32.1; no longer R30.2, R31.1
- net N$3: now also R13.2, R41.2; no longer R12.2, R39.2
- net N$31: now also R37.2, R46.1, R47.2; no longer R36.2, R45.1, R46.2
- net N$32: now also D14.C; no longer D1.C
- net N$35: now also D12.C, D13.A; no longer D17.C, D18.A
- net N$37: now also D11.C, D12.A; no longer D16.C, D17.A
- net N$38: now also D10.C, D11.A; no longer D15.C, D16.A
- net N$4: now also R12.1, R39.2; no longer R11.1, R37.2
- net N$44: now also D17.C, R35.2; no longer D24.C, R34.2
- net N$46: now also D13.C; no longer D18.C
- net N$47: now also D15.C; no longer D21.C
- net N$5: now also R24.1; no longer R23.1
- net N$6: now also R43.1; no longer R41.1
- net N$8: now also R45.1; no longer R43.1
- net PARTICLE_RST: now also ASSY1.D3, R48.1; no longer R47.1
- net SD_ENABLE: now also R29.2; no longer R28.2
- net SD_MISO: now also R18.1; no longer R17.1
- net SD_MOSI: now also R16.1; no longer R15.1
- net SENSORS_SCL: now also R19.1; no longer R18.1
- net SENSORS_SDA: now also R15.1; no longer R14.1
- net SERIAL_NUM: now also R14.2; no longer R13.2
- net TDR_L_DETECT: now also D4.C, R35.1; no longer D25.C, R34.1
- net TDR_N_DETECT: now also D3.C, R36.1; no longer D28.C, R35.1
- net VCC: now also R14.1, R15.2, R19.2, R22.1, R34.1; no longer R13.1, R14.2, R18.2, R20.1, R33.1
- net WDI: now also R20.1; no longer R19.1
Routing:
- net PARTICLE_RST: track 1.67 -> 17.0 mm
- net N$1: track 0.00 -> 3.81 mm
- net AC_SENSE_VCC: track 63.9 -> 66.7 mm
- net TDR_N_DETECT: track 84.1 -> 86.8 mm
- net REF_1V5: track 41.0 -> 43.6 mm
- net N$3: track 12.0 -> 13.9 mm
- net GND: track 8.01 -> 9.88 mm, vias 78 -> 77
- net N$6: track 12.2 -> 13.8 mm
- net N$7: track 0.00 -> 1.07 mm
- net N$17: track 5.36 -> 4.43 mm
- net TDR_N_TRIGGER: track 88.5 -> 89.3 mm
- net REF_3V: track 38.4 -> 37.6 mm
- net AC_N2: track 8.36 -> 8.88 mm
- net AC_N1: track 6.95 -> 7.46 mm
- net TDR_L_TRIGGER: track 67.3 -> 66.8 mm

Commit message: remove previous production files and TDR circuit
Parts:
- removed C12, C13: 10nF, SparkFun-Capacitors:1206
- removed C4, C5: 100pF, passives:0402_CAP
- removed C6, C7: 1nF, passives:0402_CAP
- removed D16, D17, D18, D19: 1000Vr, diode:DO214AC
- removed D3, D4: 3V, SparkFun-DiscreteSemi:SOD-323
- removed R35, R36: 806k, passives:0805_RES
- removed R4, R5: 40.2, passives:0402_RES
- removed U15, U16, U17, U18: SN74LVC1G86DRLRDRL5-L, SN74LVC1G86:DRL5-L
- moved C16 2.18 mm to (6.86, 26.9)
- moved C19 2.18 mm to (4.83, 26.9)
- moved R38 2.09 mm to (11.9, 33.8)
- moved R40 2.09 mm to (11.9, 29.7)
- moved R44 2.09 mm to (11.9, 31.5)
- moved R43 2.09 mm to (11.9, 35.6)
- moved R45 1.80 mm to (8.13, 28.8)
- moved R9 1.70 mm to (8.64, 31.2)
- moved R41 1.63 mm to (3.05, 28.8)
- moved R12 1.55 mm to (8.64, 33.5)
- moved R13 1.44 mm to (2.54, 31.0)
- moved U2 1.37 mm to (5.59, 32.4)
- moved C18 1.30 mm to (6.60, 37.3)
- moved C17 1.30 mm to (4.32, 37.3)
- moved R39 1.27 mm to (8.13, 35.7)
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Connections:
- removed net !RST1: R4.2, U15.4, U16.2
- removed net !RST2: R5.2, U17.4, U18.2
- removed net A: C4.1, R4.1, U16.1
- removed net A2: C5.1, R5.1, U18.1
- removed net AC_N1: D16.A, U16.4
- removed net AC_N2: D18.A, U18.4
- removed net N$17: C13.1, D19.C, R36.2
- removed net N$44: C12.1, D17.C, R35.2
- removed net TDR_L_DETECT: ASSY1.B2, C6.1, D4.C, R35.1, U19.13
- removed net TDR_L_TRIGGER: ASSY1.B3, U15.2, U19.12
- removed net TDR_N_DETECT: ASSY1.B4, C7.1, D3.C, R36.1, U19.11
- removed net TDR_N_TRIGGER: ASSY1.B5, U17.2, U19.10
- net AC_L_HV_OUT: now also ASSY1.A0
- net AC_L_LV_OUT: now also ASSY1.B3; no longer ASSY1.A1
- net AC_L_SENSE: no longer D16.C, D17.A
- net AC_N: no longer D18.C, D19.A
- net AC_N_HV_OUT: now also ASSY1.B4
- net AC_N_LV_OUT: now also ASSY1.B5; no longer ASSY1.A0
- net AC_SENSE_VCC: no longer U15.5, U16.5, U17.5, U18.5
- net GND: no longer C12.2, C13.2, C4.2, C5.2, C6.2, C7.2, D3.A, D4.A, U15.1, U15.3, U16.3, U17.1, U17.3, U18.3
Routing:
- net TDR_N_TRIGGER: track 89.3 -> 0.00 mm, vias 2 -> 0
- net TDR_N_DETECT: track 86.8 -> 0.00 mm, vias 2 -> 0
- net TDR_L_TRIGGER: track 66.8 -> 0.00 mm, vias 2 -> 0
- net AC_L_HV_OUT: track 19.8 -> 80.6 mm
- net TDR_L_DETECT: track 57.6 -> 0.00 mm, vias 2 -> 0
- net AC_N_HV_OUT: track 25.0 -> 82.4 mm
- net AC_SENSE_VCC: track 66.7 -> 14.9 mm, vias 6 -> 0
- net AC_L_LV_OUT: track 90.3 -> 76.7 mm
- net AC_N2: track 8.88 -> 0.00 mm
- net AC_N1: track 7.46 -> 0.00 mm
- net REF_1V5: track 43.6 -> 50.4 mm
- net N$44: track 6.01 -> 0.00 mm
- net N$17: track 4.43 -> 0.00 mm
- net N$6: track 13.8 -> 17.8 mm
- net AC_N_LV_OUT: track 83.9 -> 80.3 mm
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