File: hardware/plugwatch_G/board/plugwatch.brd (EAGLE design)
At the start: 55.7 x 95.2 mm, 123 parts, among them J1 DM3AT-SF-PEJM5, J2 TC2030-JLINK-L, Q1 MOSFET-NCHANNELSMD, Q2 NX3008PBK, U1 AB1815-T3, U10 MAX7315ATET, U11 REF2030AIDDCR, U12 SIP32510, U13 SIP32510, U14 SIP32510, U19 STM32L432KC, U2 ADA4096-4ACPZ-R7, U20 TCA9406DCUR, U21 TPS79330DBVR, U3 BGA725L6-ALT, U4 DS2401P+, U5 SAFFB1G56KB0F0A, U6 IRM-03-5V, U7 LIS2DH12, U8 MAX-M8, U9 MAX67XXMAX6749MAX67XX, X1 ABS05-32.768KHZ-T, X2 ABS07-32.768KHZ-7-T

Commit message: renaming and a few layout fixes
Parts:
- removed C30: 4.7uF, passives:0402_CAP
- removed C31, C32: 10uF, passives:0402_CAP
- removed C33, C34: 100uF, passives:1210_CAP
- removed C35: 2000uF, rcl:E5-13
- removed R45: 953k, passives:0805_RES
- removed R46, R47, R48: 1M, passives:0402_RES
- added C12, C13: 0.1uF, passives:0402_CAP
- added C4, C5, C6, C7: 10nF, passives:0402_CAP
- added R35, R36: 953k, passives:0805_RES
- added R4: 475, passives:0402_RES
- added R5: 750, passives:0402_RES
- C10, C11, C8, C9: value 10nF -> 0.1uF
- C17: value 0.1uF -> 0.82uF
- C18, C19, C20, C21: value 0.1uF -> 1uF
- C22: value 0.1uF -> 2.2uF
- C23: value 0.82uF -> 4.7uF
- C24: value 1uF -> 4.7uF
- C25, C26: value 1uF -> 10uF
- C27: value 1uF -> 100uF; device passives:0402_CAP -> passives:1210_CAP
- C28: value 2.2uF -> 100uF; device passives:0402_CAP -> passives:1210_CAP
- C29: value 4.7uF -> 2000uF; device passives:0402_CAP -> rcl:E5-13
- D29: value SML-LX0404SIUPGUSB -> (none)
- R10, R11: value 1.69k -> 3.74k
- R12: value 3.74k -> 5.1k
- R13: value 3.74k -> 10k
- R14: value 5.1k -> 10k
- R24: value 10k -> 34k
- R25: value 10k -> 66.5k
- R26: value 34k -> 100k
- R27: value 66.5k -> 100k
- R33: value 100k -> 825k
- R34: value 100k -> 953k; device passives:0402_RES -> passives:0805_RES
- R37: value 825k -> 953k; device passives:0402_RES -> passives:0805_RES
- R42, R43, R44: value 953k -> 1M; device passives:0805_RES -> passives:0402_RES
- R6: value 475 -> 1.00k
- R7: value 750 -> 1.00k
- R8, R9: value 1.00k -> 1.69k
- moved R34 63.5 mm to (11.9, 33.8), turned to 180 degrees
- moved C27 60.1 mm to (51.4, 14.6), turned to 90 degrees
- moved R8 60.0 mm to (16.3, 91.9), turned to 0 degrees
- moved R10 58.9 mm to (8.64, 33.5), turned to 270 degrees
- moved R6 58.8 mm to (2.54, 33.5), turned to 270 degrees
- moved R7 58.5 mm to (8.64, 31.2), turned to 90 degrees
- moved R12 51.4 mm to (2.41, 84.6), turned to 0 degrees
- moved C28 47.8 mm to (51.4, 20.1)
- moved C14 45.9 mm to (3.05, 46.7), turned to 180 degrees
- moved R13 44.4 mm to (20.3, 71.6), turned to 180 degrees
- moved R25 43.9 mm to (36.2, 86.7)
- moved C29 43.1 mm to (48.3, 35.9), turned to 180 degrees
- moved R37 40.0 mm to (3.05, 28.8), turned to 180 degrees
- moved R32 38.5 mm to (43.3, 89.0), turned to 270 degrees
- moved R44 37.9 mm to (35.8, 61.0), turned to 90 degrees
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- renumbered U19 to U15, U20 to U16, U21 to U17
Connections:
- net !EXTERNAL_RST: now also R21.2; no longer R23.2
- net !RTC_CS: now also R20.2; no longer R24.2
- net !RTC_INT1: now also R19.2; no longer R21.2
- net !RTC_INT2: now also R32.2; no longer R34.2
- net !SD_CS: now also R15.1; no longer R17.1
- net !SD_DETECT: now also R26.1; no longer R28.1
- net 5V: now also C27.1, C28.1, C29.+, R24.1, R29.1, R43.1; no longer C33.1, C34.1, C35.+, R26.1, R31.1, R47.1
- net AC_COPROC_VCC: now also C15.1, C16.1, C20.1, C24.1; no longer C22.1, C26.1, C27.1, C30.1
- net AC_L_800V_DETECT: now also C6.1; no longer C10.1
- net AC_L_HV_OUT: now also R6.2; no longer R8.2
- net AC_L_LV_OUT: now also R10.2; no longer R12.2
- net AC_L_SENSE: now also R34.1, R39.2; no longer R38.1, R43.2
- net AC_N: now also R36.1, R40.2; no longer R40.1, R44.2
- net AC_N_800V_DETECT: now also C7.1; no longer C11.1
- net AC_N_HV_OUT: now also R7.2; no longer R9.2
- net AC_N_LV_OUT: now also R11.1; no longer R13.1
- net AC_SENSE_PWR_EN: now also R31.2; no longer R33.2
- net BOOT0: now also R23.2; no longer R25.2
- net GND: now also C12.2, C13.2, C14.2, C26.1, C29.-, C4.1, C5.1, C6.2, C7.2, C9.2, R18.2, R23.1, R25.2, R27.1, R28.1, R30.2, R31.1, R35.1, R37.1, R38.2, R41.2, R44.2, R9.1; no longer C14.1, C26.2, C29.2, C30.2, C31.2, C32.1, C33.2, C34.2, C35.-, C9.1, R11.1, R20.2, R25.1, R27.2, R29.1, R30.1, R32.2, R33.1, R39.1, R41.1, R45.2, R46.2, R48.2
- net GPS_PWR_EN: now also R28.2; no longer R30.2
- net GPS_VCC: now also C26.2, C5.2, C8.2; no longer C14.2, C32.2, C9.2
- net N$1: now also R9.2; no longer R11.2
- net N$10: now also R24.2, R25.1; no longer R26.2, R27.1
- net N$18: now also C23.1, R14.2, R15.2, R26.2; no longer C29.1, R17.2, R18.2, R28.2
- net N$23: now also R21.1, R33.1; no longer R23.1, R37.1
- net N$25: now also R29.2, R30.1; no longer R31.2, R32.1
- net N$26: now also R4.1; no longer R6.1
- net N$3: now also R11.2, R36.2, R37.2; no longer R13.2, R40.2, R41.2
- net N$31: now also R33.2, R42.1, R43.2; no longer R37.2, R46.1, R47.2
- net N$36: now also C17.1; no longer C23.1
- net N$39: now also C22.1; no longer C28.1
- net N$4: now also R10.1, R34.2, R35.2; no longer R12.1, R38.2, R39.2
- net N$42: now also R5.1; no longer R7.1
- net N$49: now also R8.1; no longer R10.1
- net N$5: now also R22.1; no longer R24.1
- net N$50: now also R8.2; no longer R10.2
- net N$51: now also R5.2; no longer R7.2
- net N$52: now also R4.2; no longer R6.2
- net N$6: now also R38.1, R39.1, R6.1; no longer R42.1, R43.1, R8.1
- net N$8: now also R40.1, R41.1, R7.1; no longer R44.1, R45.1, R9.1
- net PARTICLE_RST: now also R44.1; no longer R48.1
- net REF_1V5: now also C10.1, C11.1, C12.1, C13.1; no longer C16.1, C17.1, C18.1, C19.1
- net REF_3V: now also C14.1, C19.1; no longer C20.1, C25.1
- net SD_ENABLE: now also R27.2; no longer R29.2
- net SD_MISO: now also R16.1; no longer R18.1
- net SD_MOSI: now also R14.1; no longer R16.1
- net SENSORS_SCL: now also R17.1; no longer R19.1
- net SENSORS_SDA: now also R13.1; no longer R15.1
- net SERIAL_NUM: now also R12.2; no longer R14.2
- net VCC: now also C18.1, C25.1, C9.1, R12.1, R13.2, R17.2, R19.1, R20.1, R32.1; no longer C15.1, C24.1, C31.1, R14.1, R15.2, R19.2, R21.1, R22.1, R34.1
- net VCC_RF: now also C4.2; no longer C8.2
- net WDI: now also R18.1; no longer R20.1
