File: hardware/plugwatch_G/board/plugwatch.sch (EAGLE design)
At the start: 125 parts, among them J1 DM3AT-SF-PEJM5, J2 SCREW_TERMNIAL_1, J3 SCREW_TERMNIAL_1, U1 AB1815-T3, U10 OPA369, U11 SIP32510, U12 SIP32510, U13 SIP32510, U14 SIP32510, U2 BGA725L6-ALT, U3 DS2401P+, U4 SAFFB1G56KB0F0A, U5 IRM-03-5V, U6 LIS2DH12, U7 MAX-M8, U8 MAX67XXMAX6749MAX67XX, U9 OPA369, X1 ABS07-32.768KHZ-7-T

Commit message: update board and schematic with changes from last revision
Parts:
- removed ASSY2: WRL-13678, chips:WRL-13678
- removed C11: 1uF, passives:CAPACITOR0402_CAP
- removed D5: BLUE, leds:LED0603
- removed R23: 100k, passives:RESISTOR0402_RES
- removed R4: 68, passives:RESISTOR0402_RES
- removed R5: 1k, passives:RESISTOR0402_RES
- removed TP1, TP2, TP20, TP21, TP22, TP3: TEST_POINT_0.040IN, headers:TEST_POINT_0.040IN
- removed U13: SIP32510, chips:SIP32510
- removed U15: (no value), microphones:SPH0645LM4H-B
- added Q1: NX3008PBK, fets:NX3008PBK
- added Q2: MOSFET-NCHANNELSMD, fets:MOSFET-NCHANNELSMD
- R1: value 66.5 -> 66.5K
- R2: value 68 -> 100k; DESCRIPTION RES SMD 68 OHM 1% 1/16W 0402 -> RES SMD 34K OHM 1% 1/10W 0402; DIGIKEY 311-68.0LRCT-ND -> P34.0KLCT-ND; MANUFACTURER Yageo -> Panasonic Electronic Components; MPN RC0402FR-0768RL -> ERJ-2RKF3402X
- R27: value 499k -> 1M
- R3: value 68 -> 1M; DESCRIPTION RES SMD 68 OHM 1% 1/16W 0402 -> RES SMD 499K OHM 1% 1/10W 0402; DIGIKEY 311-68.0LRCT-ND -> P499KLCT-ND; MANUFACTURER Yageo -> Panasonic Electronic Components; MPN RC0402FR-0768RL -> ERJ-2RKF4993X
Connections:
- removed net MIC_BCLK: ASSY1.D4, R3.2, TP22.TESTPOINT
- removed net MIC_DATA: ASSY1.D2, R4.1, TP21.TESTPOINT
- removed net MIC_WS: ASSY1.D5, R2.2, TP20.TESTPOINT
- removed net N$1: D5.ANODE, R5.1
- removed net N$12: R3.1, U15.BCLK
- removed net N$14: ASSY2.!RST, ASSY2.3V3, ASSY2.EN, U13.VLOAD
- removed net N$15: R4.2, U15.DATA
- removed net N$2: D5.CATHODE, U7.TIMEPULSE
- removed net N$3: R2.1, U15.WS
- removed net WIFI_PWR_EN: ASSY1.B1, R23.2, TP1.TESTPOINT, U13.EN
- removed net WIFI_RXD: ASSY1.C1, ASSY2.RXI, TP3.TESTPOINT
- removed net WIFI_TXD: ASSY1.C0, ASSY2.TXO, TP2.TESTPOINT
- new net !RTC_INT2: ASSY1.D2, Q1.G, R2.2, U1.!IRQ2
- new net DO_NOT_CONNECT: ASSY1.D7
- new net GPS_PPS: ASSY1.D4, U7.TIMEPULSE
- new net PARTICLE_RST: Q2.G, R3.1
- net !RTC_INT1: now also ASSY1.D5; no longer ASSY1.D7
- net GND: now also Q2.S, R3.2; no longer ASSY2.GND, C11.2, R23.1, U13.GND, U15.GND
- net GPS_VCC: no longer R5.2
- net N$10: now also Q1.D
- net N$31: now also Q2.D
- net VCC: now also Q1.S, R2.1; no longer C11.1, U13.VSUPP, U15.SELECT, U15.VDD
Other:
- note added: "The RTC exposes only open drain interrupts, but the particle only wakes up on a rising edge. The idea here is that once the RTC_INT2 pulls down it will activate the PFET pulling up the WKP pin. IF the power turns on the PFET is effectively off, and the WKP net is still floating so that the 5V signal can pull it up."
- note added: "Voltage supervisor. MR is the voltage input. MR Triggers below 1.235V. We want reset if: (Batt < 3.3v AND !5V) OR PARTICLE_RST Current circuit: If PARTICLE_RST = 1, MR=0 If Bat = 3.3 and 5V=0 then MR=1.235, If bat = 0 and 5V = 5V then MR = 1.556."
- note removed: "Voltage supervisor. MR is the voltage input. MR Triggers at 1.235V. We want to trigger at 3.3V, so voltage divide down with 1% resistors."
- note removed: "WiFi"
- note removed: "https://cdn.sparkfun.com/datasheets/Wireless/WiFi/ESP8266ModuleV1.pdf"
- moved on the sheet: ASSY1, R1, R19

Commit message: add new voltage amplifier circuit
Parts:
- removed D1, D2, D3, D4: (no value), passives:DIODE_ZENERSOT323
- removed R37, R38, R39, R40: 1M, passives:RESISTOR0402_RES
- removed U10, U9: OPA369, powerfilm:OPA369
- added C11, C18: 0.1uF, passives:CAPACITOR0402_CAP
- added R23: 953k, passives:RESISTOR0402_RES
- added R4: 1, resistor:R-US_R2512
- added R5: 3.74k, passives:RESISTOR0402_RES
- added U13: ADA4096-4ACPZ-R7, ada4096-4:ADA4096-4ACPZ-R7
- added U15: REF2033AIDDCR, ref2033:REF2033AIDDCR
- R28, R30, R31: value 750k -> 953k; device passives:RESISTOR1206_RES_HIGH_CLEARANCE -> passives:RESISTOR0402_RES; DESCRIPTION RES SMD 750K OHM 1% 1/4W 1206 -> RES SMD 100K OHM 1% 1/16W 0402; DIGIKEY 311-750KFRCT-ND -> 541-100KLCT-ND; MANUFACTURER Yageo -> Vishay Dale; MPN RC1206FR-07750KL -> CRCW0402100KFKED
- R29: value 750k -> 3.75k; device passives:RESISTOR1206_RES_HIGH_CLEARANCE -> passives:RESISTOR0402_RES; DESCRIPTION RES SMD 750K OHM 1% 1/4W 1206 -> RES SMD 100K OHM 1% 1/16W 0402; DIGIKEY 311-750KFRCT-ND -> 541-100KLCT-ND; MANUFACTURER Yageo -> Vishay Dale; MPN RC1206FR-07750KL -> CRCW0402100KFKED
- R33: value 953k -> 1.00k; DESCRIPTION RES SMD 953K OHM 1% 1/16W 0402 -> RES SMD 100K OHM 1% 1/16W 0402; DIGIKEY YAG3262CT-ND -> 541-100KLCT-ND; MANUFACTURER Yageo -> Vishay Dale; MPN RC0402FR-07953KL -> CRCW0402100KFKED
- R34: DESCRIPTION RES SMD 953K OHM 1% 1/16W 0402 -> RES SMD 100K OHM 1% 1/16W 0402; DIGIKEY YAG3262CT-ND -> 541-100KLCT-ND; MANUFACTURER Yageo -> Vishay Dale; MPN RC0402FR-07953KL -> CRCW0402100KFKED
- R35: device passives:RESISTOR1206_RES_HIGH_CLEARANCE -> passives:RESISTOR0402_RES; DESCRIPTION (none) -> RES SMD 100K OHM 1% 1/16W 0402; DIGIKEY P953KBCCT-ND -> 541-100KLCT-ND; MANUFACTURER Panasonic Electronic Components -> Vishay Dale; MPN ERA-8AEB9533V -> CRCW0402100KFKED
- R36: value 953k -> 1.00k; device passives:RESISTOR1206_RES_HIGH_CLEARANCE -> passives:RESISTOR0402_RES; DESCRIPTION (none) -> RES SMD 100K OHM 1% 1/16W 0402; DIGIKEY P953KBCCT-ND -> 541-100KLCT-ND; MANUFACTURER Panasonic Electronic Components -> Vishay Dale; MPN ERA-8AEB9533V -> CRCW0402100KFKED
- R6, R7: value 4.99k -> 953k; DESCRIPTION RES SMD 4.99K OHM 1% 1/10W 0402 -> RES SMD 100K OHM 1% 1/16W 0402; DIGIKEY P4.99KLCT-ND -> 541-100KLCT-ND; MANUFACTURER Panasonic Electronic Components -> Vishay Dale; MPN ERJ-2RKF4991X -> CRCW0402100KFKED
Connections:
- removed net AC/L-FUSED: F1.P$2, R28.1, R30.1, R35.1, U5.AC/L, V1.1
- removed net AC/N-FUSED: J3.P$1, R29.1, R31.1, R36.1, U5.AC/N, V1.2
- removed net N$38: F1.P$1, J2.P$1
- removed net N$42: R37.1, R38.2, U9.IN+
- removed net N$43: R33.2, R35.2, R6.1, U9.IN-
- removed net N$44: R39.1, R40.2, U10.IN+
- removed net N$45: R34.2, R36.2, R7.1, U10.IN-
- removed net SENSE_VCC: C5.1, C6.1, R37.2, R39.2, U10.VCC, U14.VLOAD, U9.VCC
- new net AC_L_HV_OUT: R33.2, U13.OUTC
- new net AC_L_LV_OUT: R5.2, U13.OUTA
- new net AC_L_SENSE: F1.P$1, J2.P$1, R31.2, R6.1
- new net AC_N: J3.P$1, R23.1, R34.2, U5.AC/N, V1.2
- new net AC_N_HV_OUT: R36.2, U13.OUTD
- new net AC_N_LV_OUT: R29.1, U13.OUTB
- new net AC_SENSE_VCC: U14.VLOAD, U15.EN, U15.VIN
- new net N$1: F1.P$2, R4.1
- new net N$2: R4.2, U5.AC/L, V1.1
- new net N$3: R23.2, R28.2, R29.2, U13.-INB
- new net N$4: R5.1, R6.2, R7.2, U13.-INA
- new net N$6: R30.1, R31.1, R33.1, U13.-INC
- new net N$8: R34.1, R35.1, R36.1, U13.-IND
- new net REF_1V65: C11.1, C18.1, C5.1, C6.1, U13.+INA, U13.+INB, U13.+INC, U13.+IND, U15.VBIAS
- new net REF_3V3: U13.V+, U15.VREF
- net AC/L-MEASURE: no longer D1.CATHODE, R30.2
- net AC/L-PERTURB: no longer D2.CATHODE, R28.2
- net AC/L-SENSE: no longer R6.2, U9.OUT
- net AC/N-MEASURE: no longer D3.CATHODE, R31.2
- net AC/N-PERTURB: no longer D4.CATHODE, R29.2
- net AC/N-SENSE: no longer R7.2, U10.OUT
- net GND: now also C11.2, C18.2, R28.1, R30.2, R35.2, R7.1, U13.-V, U13.EP, U15.GND; no longer D1.ANODE, D2.ANODE, D3.ANODE, D4.ANODE, R33.1, R34.1, R38.1, R40.1, U10.VSS, U9.VSS
Other:
- note added: "There are two goals of the sensing circuit: 1) be able to sense voltages precisely from 0-340vpp and less precisely from 340-1500vpp. 2) Protect the AC/DC converter which has a maximum voltage of 280vac rms. The theory of operation here is that in normal mode the MOV isn't conducting, current through R4 is rather low, and it's power dissipation is also low. In a voltage spike scenario the MOV wil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"
- note added: "This op amp has built in over voltage protection, so while op-amps A and B experience > 3.3V on their input in high voltage scenarios the op amp is made to handle that."
- note added: "This ref supplies 20ma at low (300mv) drop out. We can use it to supply VDDA of the MCU, the Amps and bias the non-inverting side of the amps. Using the same source for all of this should eliminate many sources of noise."
- note removed: "-(RF/RI)*VTEST + VCC/2"
- note removed: "3.3V Zener Diode"
- note removed: "Assuming 340Vpp, a 750k resistor will dissipate 0.15W, and a 3.3v zener will dissipate 1.4mW"
- note removed: "Output voltage:"
- note removed: "The schottkey diode is necessary to protect the MCU pin against the -0.7-1V potentially caused by the zener forward voltage if AC/L or AC/N are negative relative to GND. The schottkey has Vf < 0.3 which is less than the internal diodes on most MCUs."
- note removed: "This circuit handles up to 340V with a 3.3V reference."
- note removed: "We use a seperate AC Measure pin so that we can more directly sense the perturbation by the digital output. The full-scale voltage sensing circuit (below) could also be used, but would only sense <1% of its dynamic range."
- moved on the sheet: C15, C16, C17, C5, C6, F1, J2, J3, R26, R28, R29, R30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

Commit message: finish up direct voltage sensing, add coprocessor and i2c translator
Parts:
- added C19, C21: 0.1uF, passives:CAPACITOR0402_CAP
- added C20, C22: 1uF, passives:CAPACITOR0402_CAP
- added C23: 4.7uF, passives:CAPACITOR0402_CAP
- added C24, C25: 4.3pF, passives:CAPACITOR0402_CAP
- added J4: TC2030-JLINK-L, connector:TC2030-JLINK-L
- added R37: 10k, passives:RESISTOR0402_RES
- added S1: B3U-1000P, switches:B3U-1000P
- added U10: STM32L432KC, chips:STM32L432KC
- added U16: TCA9406DCUR, tca9406:TCA9406DCUR
- added U9: TPS79330DBVR, tps7933:TPS79330DBVR
- added X2: ABS05-32.768KHZ-T, crystals:ABS05-32.768KHZ-T
- U15: value REF2033AIDDCR -> REF2030AIDDCR; MANUFACTURER_PART_NUMBER (none) -> REF2030AIDDCR
Connections:
- net REF_1V65 renamed REF_1V5
- removed net REF_3V3: U13.V+, U15.VREF
- new net !RST: J4.!RESET, R37.2, S1.P$2, U10.!RST, U10.PH3/BOOT0
- new net AC_COPROC_VCC: C21.1, C22.1, C23.1, J4.VCC, U10.VDD, U16.OE, U16.VCCA, U9.OUT
- new net AC_SCL: U10.PA9, U16.SCL_A
- new net AC_SDA: U10.PA10, U16.SDA_A
- new net N$11: C24.2, U10.PC14/OSC32IN, X2.2
- new net N$9: C25.2, U10.PC15/OSC32OUT, X2.1
- new net REF_3V: C19.1, C20.1, U10.VDDA/VREF, U13.V+, U15.VREF
- new net SWDCLK: J4.SWDCLK, U10.PA14/SWDCLK
- new net SWDIO: J4.SWDIO, U10.PA13/SWDIO
- net AC_L_HV_OUT: now also U10.PA2
- net AC_L_LV_OUT: now also U10.PA0/CLKIN
- net AC_N_HV_OUT: now also U10.PA3
- net AC_N_LV_OUT: now also U10.PA1
- net AC_SENSE_VCC: now also U9.EN, U9.IN
- net GND: now also C19.2, C20.2, C21.2, C22.2, C23.2, C24.1, C25.1, J4.GND, R37.1, S1.P$1, U10.VSS, U16.GND, U9.GND
- net SENSORS_SCL: now also U16.SCL_B
- net SENSORS_SDA: now also U16.SDA_B
- net VCC: now also U16.VCCB
Other:
- note added: "REGULATE 3V3 to 3V so that VDDA can be powered by the reference."
- note removed: "GPS and WiFi Radios"

Commit message: add TDR, connect PPS, add transient spike detectors
Parts:
- added C26, C27, C28, C29: 0.01uF, passives:CAPACITOR0402_CAP
- added C30, C33: 100pF, passives:CAPACITOR0402_CAP
- added C31, C32, C34, C35: 10nF, passives:CAPACITOR0402_CAP
- added D1, D2, D21, D22, D23, D26: 2000Vr, diode:DIODE-DO214AC
- added D10, D11, D19, D20, D25, D28: 3V, SparkFun-DiscreteSemi:DIODE-ZENER-MM3Z3V3T1G
- added D12, D13, D14, D15, D16, D17, D18, D3, D4, D5, D6, D7, D8, D9: 200V, diode:DIODE-DO214AA
- added D24, D27: >1kVr, diode:DIODE-DO214AC
- added R38, R39, R40, R42: 10, passives:RESISTOR0402_RES
- added R43, R46: 40, passives:RESISTOR0402_RES
- added R44, R47: 800k, passives:RESISTOR0402_RES
- added R45, R48: 1M, passives:RESISTOR0402_RES
- added U17, U18, U21, U22: SN74LVC1G86DBVR, SN74LVC:SN74LVC1G86DBVR
Connections:
- new net !RST1: R43.2, U21.Y, U22.B
- new net !RST2: R46.2, U17.Y, U18.B
- new net AC_L_600V_DETECT: C27.1, D11.C, D4.A, U10.PB5
- new net AC_L_800V_DETECT: C26.1, D10.C, D6.A, U10.PB4/!JTRST
- new net AC_N1: D23.A, U22.Y
- new net AC_N2: D26.A, U18.Y
- new net AC_N_600V_DETECT: C29.1, D13.A, D20.C, U10.PB7
- new net AC_N_800V_DETECT: C28.1, D15.A, D19.C, U10.PB6
- new net GND1: C30.1, R43.1, U22.A
- new net GND2: C33.1, R46.1, U18.A
- new net N$12: F1.P$1, J2.P$1
- new net N$14: D8.C, D9.A
- new net N$15: D7.C, D8.A
- new net N$16: D6.C, D7.A
- new net N$17: C34.1, D27.C, R47.2
- new net N$22: D5.C, R39.1
- new net N$24: D3.A, D4.C
- new net N$30: D9.C, R38.1
- new net N$32: D1.C, R38.2
- new net N$33: D2.C, R39.2
- new net N$34: D12.C, D14.A
- new net N$35: D17.C, D18.A
- new net N$37: D16.C, D17.A
- new net N$38: D15.C, D16.A
- new net N$43: D12.A, D13.C
- new net N$44: C31.1, D24.C, R44.2
- new net N$45: D14.C, R42.1
- new net N$46: D18.C, R40.1
- new net N$47: D21.C, R40.2
- new net N$48: D22.C, R42.2
- new net TDR_L_DETECT: C32.1, D25.C, R44.1, R45.2, U10.PA4
- new net TDR_L_TRIGGER: U10.PA6, U21.B
- new net TDR_N_DETECT: C35.1, D28.C, R47.1, R48.2, U10.PA5
- new net TDR_N_TRIGGER: U10.PA7, U17.B
- net AC_L_SENSE: now also D1.A, D2.A, D23.C, D24.A, F1.P$2, R4.1; no longer F1.P$1, J2.P$1
- net AC_N: now also D21.A, D22.A, D26.C, D27.A
- net AC_SENSE_VCC: now also U17.VCC, U18.VCC, U21.VCC, U22.VCC
- net GND: now also C26.2, C27.2, C28.2, C29.2, C30.2, C31.2, C32.2, C33.2, C34.2, C35.2, D10.A, D11.A, D19.A, D20.A, D25.A, D28.A, R45.1, R48.1, U17.A, U17.GND, U18.GND, U21.A, U21.GND, U22.GND
- net GPS_PPS: now also U10.PB3/JTDO/SWO
- net N$1: now also D3.C, D5.A; no longer F1.P$2, R4.1
Other:
- note added: "The pulse response can up to double. We want to sense this impulse overlap (voltage increase) so we need a divider circuit. Zener protects the pin from overvoltage while AC is on. Capacitor allows for better ADC sampling due to high source impedance."
- note added: "This circuit generates a pulse of ~4ns (modulo non-linear time delays). If the wire is shorter than a 4ns pulse time, the reflected voltage will be higher than the input voltage (3V3 - Vfr of the diode). If it's longer then it will not increase. 4ns should be 50-150cm depending on the wire and insulation."
- note added: "This diode protects the output of the XOR. As low of drop as possible, very high Vr."
- note added: "This is a sample and hold circuit. C needs to withstand AC voltages, D needs to have high Vr and low drop."
- note removed: "This will protect the sampling circuit against surges"

Commit message: split the symbol up for the op amp so it's readable
Parts:
- R29: value 3.75k -> 3.74k
Connections:
- net AC_L_HV_OUT: now also U13D.OUT; no longer U13.OUTC
- net AC_L_LV_OUT: now also U13C.OUT; no longer U13.OUTA
- net AC_N_HV_OUT: now also U13B.OUT; no longer U13.OUTD
- net AC_N_LV_OUT: now also U13A.OUT; no longer U13.OUTB
- net GND: now also U13SUPPLY.V-; no longer U13.-V, U13.EP
- net N$3: now also U13A.-; no longer U13.-INB
- net N$4: now also U13C.-; no longer U13.-INA
- net N$6: now also U13D.-; no longer U13.-INC
- net N$8: now also U13B.-; no longer U13.-IND
- net REF_1V5: now also U13A.+, U13B.+, U13C.+, U13D.+; no longer U13.+INA, U13.+INB, U13.+INC, U13.+IND
- net REF_3V: now also U13SUPPLY.V+; no longer U13.V+
Other:
- moved on the sheet: C11, C18, C5, C6, R23, R26, R28, R29, R30, R31, R33, R34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
