File: hardware/plugwatch_G/board/plugwatch.sch (EAGLE design)
At the start: 176 parts, among them J1 DM3AT-SF-PEJM5, J2 SCREW_TERMNIAL_1, J3 SCREW_TERMNIAL_1, J4 TC2030-JLINK-L, Q1 NX3008PBK, Q2 MOSFET-NCHANNELSMD, U1 AB1815-T3, U10 STM32L432KC, U11 SIP32510, U12 SIP32510, U13 ADA4096-4ACPZ-R7, U14 SIP32510, U15 REF2030AIDDCR, U16 TCA9406DCUR, U17 SN74LVC1G86DBVR, U18 SN74LVC1G86DBVR, U2 BGA725L6-ALT, U21 SN74LVC1G86DBVR, U22 SN74LVC1G86DBVR, U3 DS2401P+, U4 SAFFB1G56KB0F0A, U5 IRM-03-5V, U6 LIS2DH12, U7 MAX-M8, U8 MAX67XXMAX6749MAX67XX, U9 TPS79330DBVR, X1 ABS07-32.768KHZ-7-T, X2 ABS05-32.768KHZ-T

Commit message: add new plugwatch stuff
Parts:
- removed R45, R48: 1M, passives:RESISTOR0402_RES
- C32, C35: value 10nF -> 1nF
Connections:
- net GND: no longer R45.1, R48.1
- net TDR_L_DETECT: no longer R45.2
- net TDR_N_DETECT: no longer R48.2
Other:
- moved on the sheet: D25, D28
Changed lines of the file:
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@@
 <attribute name="MPN" value="CRCW0402100KFKED"/>
 </part>
-<part name="R45" library="passives" deviceset="RESISTOR" device="0402_RES" value="1M">
-<attribute name="DESCRIPTION" value="RES SMD 100K OHM 1% 1/16W 0402"/>
-<attribute name="DIGIKEY" value="541-100KLCT-ND"/>
-<attribute name="MANUFACTURER" value="Vishay Dale"/>
-<attribute name="MPN" value="CRCW0402100KFKED"/>
-</part>
-<part name="SUPPLY30" library="umich" deviceset="GND" device=""/>
-<part name="C32" library="passives" deviceset="CAPACITOR" device="0402_CAP" value="10nF">
+<part name="C32" library="passives" deviceset="CAPACITOR" device="0402_CAP" value="1nF">
 <attribute name="DESCRIPTION" value="CAP CER 0.1UF 10V X5R 0402"/>
 <attribute name="DIGIKEY" value="311-1336-1-ND"/>
@@
 <attribute name="MPN" value="CRCW0402100KFKED"/>
 </part>
-<part name="R48" library="passives" deviceset="RESISTOR" device="0402_RES" value="1M">
-<attribute name="DESCRIPTION" value="RES SMD 100K OHM 1% 1/16W 0402"/>
-<attribute name="DIGIKEY" value="541-100KLCT-ND"/>
-<attribute name="MANUFACTURER" value="Vishay Dale"/>
-<attribute name="MPN" value="CRCW0402100KFKED"/>
-</part>
-<part name="SUPPLY39" library="umich" deviceset="GND" device=""/>
-<part name="C35" library="passives" deviceset="CAPACITOR" device="0402_CAP" value="10nF">
+<part name="C35" library="passives" deviceset="CAPACITOR" device="0402_CAP" value="1nF">
 <attribute name="DESCRIPTION" value="CAP CER 0.1UF 10V X5R 0402"/>
 <attribute name="DIGIKEY" value="311-1336-1-ND"/>
@@
 <attribute name="VALUE" x="181.102" y="123.19" size="1.778" layer="96" rot="R90"/>
 </instance>
-<instance part="R45" gate="G$1" x="177.8" y="114.3" smashed="yes" rot="R90">
-<attribute name="DIGIKEY" x="177.8" y="114.3" size="1.27" layer="96" font="vector" rot="R90" display="off"/>
-<attribute name="NAME" x="176.3014" y="110.49" size="1.778" layer="95" rot="R90"/>
-<attribute name="VALUE" x="181.102" y="110.49" size="1.778" layer="96" rot="R90"/>
-</instance>
-<instance part="SUPPLY30" gate="1" x="177.8" y="104.14" smashed="yes">
-<attribute name="VALUE" x="175.26" y="101.6" size="1.778" layer="96"/>
-</instance>
 <instance part="C32" gate="G$1" x="198.12" y="114.3" smashed="yes">
 <attribute name="DIGIKEY" x="198.12" y="114.3" size="1.016" layer="96" rot="R270" align="bottom-center" display="off"/>
@@
 <attribute name="VALUE" x="195.58" y="101.6" size="1.778" layer="96"/>
 </instance>
-<instance part="D25" gate="G$1" x="187.96" y="111.76" smashed="yes" rot="R90">
-<attribute name="NAME" x="185.928" y="109.22" size="1.778" layer="95" font="vector" rot="R90"/>
-<attribute name="VALUE" x="189.992" y="109.22" size="1.778" layer="96" font="vector" rot="R90" align="top-left"/>
-</instance>
-<instance part="SUPPLY33" gate="1" x="187.96" y="104.14" smashed="yes">
-<attribute name="VALUE" x="185.42" y="101.6" size="1.778" layer="96"/>
+<instance part="D25" gate="G$1" x="177.8" y="114.3" smashed="yes" rot="R90">
+<attribute name="NAME" x="175.768" y="111.76" size="1.778" layer="95" font="vector" rot="R90"/>
+<attribute name="VALUE" x="179.832" y="111.76" size="1.778" layer="96" font="vector" rot="R90" align="top-left"/>
+</instance>
+<instance part="SUPPLY33" gate="1" x="177.8" y="104.14" smashed="yes">
+<attribute name="VALUE" x="175.26" y="101.6" size="1.778" layer="96"/>
 </instance>
 <instance part="U17" gate="A" x="30.48" y="68.58" smashed="yes" rot="MR180">
@@
 <attribute name="VALUE" x="183.642" y="49.53" size="1.778" layer="96" rot="R90"/>
 </instance>
-<instance part="R48" gate="G$1" x="180.34" y="40.64" smashed="yes" rot="R90">
-<attribute name="DIGIKEY" x="180.34" y="40.64" size="1.27" layer="96" font="vector" rot="R90" display="off"/>
-<attribute name="NAME" x="178.8414" y="36.83" size="1.778" layer="95" rot="R90"/>
-<attribute name="VALUE" x="183.642" y="36.83" size="1.778" layer="96" rot="R90"/>
-</instance>
-<instance part="SUPPLY39" gate="1" x="180.34" y="30.48" smashed="yes">
-<attribute name="VALUE" x="177.8" y="27.94" size="1.778" layer="96"/>
-</instance>
 <instance part="C35" gate="G$1" x="200.66" y="40.64" smashed="yes">
 <attribute name="DIGIKEY" x="200.66" y="40.64" size="1.016" layer="96" rot="R270" align="bottom-center" display="off"/>
@@
 <attribute name="VALUE" x="198.12" y="27.94" size="1.778" layer="96"/>
 </instance>
-<instance part="D28" gate="G$1" x="190.5" y="38.1" smashed="yes" rot="R90">
-<attribute name="NAME" x="188.468" y="35.56" size="1.778" layer="95" font="vector" rot="R90"/>
-<attribute name="VALUE" x="192.532" y="35.56" size="1.778" layer="96" font="vector" rot="R90" align="top-left"/>
-</instance>
-<instance part="SUPPLY41" gate="1" x="190.5" y="30.48" smashed="yes">
-<attribute name="VALUE" x="187.96" y="27.94" size="1.778" layer="96"/>
+<instance part="D28" gate="G$1" x="180.34" y="38.1" smashed="yes" rot="R90">
+<attribute name="NAME" x="178.308" y="35.56" size="1.778" layer="95" font="vector" rot="R90"/>
+<attribute name="VALUE" x="182.372" y="38.1" size="1.778" layer="96" font="vector" rot="R90" align="top-left"/>
+</instance>
+<instance part="SUPPLY41" gate="1" x="180.34" y="30.48" smashed="yes">
+<attribute name="VALUE" x="177.8" y="27.94" size="1.778" layer="96"/>
 </instance>
 </instances>
@@
 </segment>
 <segment>
-<pinref part="SUPPLY30" gate="1" pin="GND"/>
-<pinref part="R45" gate="G$1" pin="1"/>
-<wire x1="177.8" y1="106.68" x2="177.8" y2="109.22" width="0.1524" layer="91"/>
-</segment>
-<segment>
 <pinref part="D25" gate="G$1" pin="A"/>
-<wire x1="187.96" y1="109.22" x2="187.96" y2="106.68" width="0.1524" layer="91"/>
+<wire x1="177.8" y1="111.76" x2="177.8" y2="106.68" width="0.1524" layer="91"/>
 <pinref part="SUPPLY33" gate="1" pin="GND"/>
 </segment>
@@
 </segment>
 <segment>
-<pinref part="SUPPLY39" gate="1" pin="GND"/>
-<pinref part="R48" gate="G$1" pin="1"/>
-<wire x1="180.34" y1="33.02" x2="180.34" y2="35.56" width="0.1524" layer="91"/>
-</segment>
-<segment>
 <pinref part="D28" gate="G$1" pin="A"/>
-<wire x1="190.5" y1="35.56" x2="190.5" y2="33.02" width="0.1524" layer="91"/>
+<wire x1="180.34" y1="35.56" x2="180.34" y2="33.02" width="0.1524" layer="91"/>
 <pinref part="SUPPLY41" gate="1" pin="GND"/>
 </segment>
@@
 <segment>
 <pinref part="D25" gate="G$1" pin="C"/>
-<wire x1="187.96" y1="114.3" x2="187.96" y2="119.38" width="0.1524" layer="91"/>
-<pinref part="R45" gate="G$1" pin="2"/>
+<wire x1="177.8" y1="116.84" x2="177.8" y2="119.38" width="0.1524" layer="91"/>
 <pinref part="R44" gate="G$1" pin="1"/>
-<wire x1="177.8" y1="116.84" x2="177.8" y2="119.38" width="0.1524" layer="91"/>
 <wire x1="177.8" y1="119.38" x2="177.8" y2="121.92" width="0.1524" layer="91"/>
-<wire x1="187.96" y1="119.38" x2="177.8" y2="119.38" width="0.1524" layer="91"/>
-<junction x="177.8" y="119.38"/>
 <pinref part="C32" gate="G$1" pin="1"/>
 <wire x1="198.12" y1="116.84" x2="198.12" y2="119.38" width="0.1524" layer="91"/>
-<wire x1="198.12" y1="119.38" x2="187.96" y2="119.38" width="0.1524" layer="91"/>
-<junction x="187.96" y="119.38"/>
+<wire x1="198.12" y1="119.38" x2="177.8" y2="119.38" width="0.1524" layer="91"/>
+<junction x="177.8" y="119.38"/>
 <wire x1="198.12" y1="119.38" x2="203.2" y2="119.38" width="0.1524" layer="91"/>
 <junction x="198.12" y="119.38"/>
@@
 <segment>
 <pinref part="D28" gate="G$1" pin="C"/>
-<wire x1="190.5" y1="40.64" x2="190.5" y2="45.72" width="0.1524" layer="91"/>
-<pinref part="R48" gate="G$1" pin="2"/>
+<wire x1="180.34" y1="40.64" x2="180.34" y2="45.72" width="0.1524" layer="91"/>
 <pinref part="R47" gate="G$1" pin="1"/>
-<wire x1="180.34" y1="43.18" x2="180.34" y2="45.72" width="0.1524" layer="91"/>
 <wire x1="180.34" y1="45.72" x2="180.34" y2="48.26" width="0.1524" layer="91"/>
-<wire x1="190.5" y1="45.72" x2="180.34" y2="45.72" width="0.1524" layer="91"/>
-<junction x="180.34" y="45.72"/>
 <pinref part="C35" gate="G$1" pin="1"/>
 <wire x1="200.66" y1="43.18" x2="200.66" y2="45.72" width="0.1524" layer="91"/>
-<wire x1="200.66" y1="45.72" x2="190.5" y2="45.72" width="0.1524" layer="91"/>
-<junction x="190.5" y="45.72"/>
+<wire x1="200.66" y1="45.72" x2="180.34" y2="45.72" width="0.1524" layer="91"/>
+<junction x="180.34" y="45.72"/>
 <wire x1="200.66" y1="45.72" x2="205.74" y2="45.72" width="0.1524" layer="91"/>
 <junction x="200.66" y="45.72"/>

Commit message: add LED with intensity driver to PW, start looking at layout
Parts:
- removed J2, J3: SCREW_TERMNIAL_1, connector:SCREW_TERMNIAL_1
- removed TP10, TP11, TP12, TP13, TP14, TP15, TP16, TP17, TP18, TP19, TP23, TP24, TP25, TP26, TP27, TP28, TP29, TP30, TP31, TP32, TP4, TP5, TP6, TP7, TP8, TP9: TEST_POINT_0.040IN, headers:TEST_POINT_0.040IN
- added D29: SML-LX0404SIUPGUSB, leds:SML-LX0404SIUPGUSB
- added R45: 1.68k, passives:RESISTOR0402_RES
- added R48: 750, passives:RESISTOR0402_RES
- added R49: 474, passives:RESISTOR0402_RES
- added TP1, TP2: TEST_POINT_0.040IN, headers:TEST_POINT_0.040IN
- added U19: MAX7315ATET, MAX7315ATET:MAX7315ATET
Connections:
- removed net AC/L-MEASURE: ASSY1.B5, TP29.TESTPOINT
- removed net AC/L-PERTURB: ASSY1.A0, TP27.TESTPOINT
- removed net AC/L-SENSE: ASSY1.B4, TP31.TESTPOINT
- removed net AC/N-MEASURE: ASSY1.B3, TP28.TESTPOINT
- removed net AC/N-PERTURB: ASSY1.A1, TP32.TESTPOINT
- removed net AC/N-SENSE: ASSY1.B2, TP30.TESTPOINT
- new net N$26: D29.B, R49.1
- new net N$42: D29.G, R48.1
- new net N$49: D29.R, R45.1
- new net N$50: R45.2, U19.P0
- new net N$51: R48.2, U19.P2
- new net N$52: R49.2, U19.P1
- net !EXTERNAL_RST: no longer TP26.TESTPOINT
- net !RTC_CS: no longer TP23.TESTPOINT
- net !RTC_INT1: no longer TP24.TESTPOINT
- net !SD_CS: no longer TP18.TESTPOINT
- net !SD_DETECT: no longer TP11.TESTPOINT
- net ACCEL_INT: no longer TP8.TESTPOINT
- net AC_L_800V_DETECT: now also ASSY1.B5
- net AC_L_LV_OUT: now also ASSY1.A1
- net AC_N: now also TP2.TESTPOINT; no longer J3.P$1
- net AC_N_800V_DETECT: now also ASSY1.B4
- net AC_N_LV_OUT: now also ASSY1.A0
- net AC_SENSE_PWR_EN: no longer TP10.TESTPOINT
- net GND: now also U19.EPAD, U19.GND; no longer TP12.TESTPOINT
- net GPS_PWR_EN: now also ASSY1.C0; no longer ASSY1.D3, TP9.TESTPOINT
- net GPS_RXD: no longer TP6.TESTPOINT
- net GPS_TXD: no longer TP14.TESTPOINT
- net N$12: now also TP1.TESTPOINT; no longer J2.P$1
- net SD_ENABLE: no longer TP19.TESTPOINT
- net SD_MISO: no longer TP16.TESTPOINT
- net SD_MOSI: no longer TP15.TESTPOINT
- net SD_SCLK: no longer TP17.TESTPOINT
- net SENSORS_SCL: now also U19.SCL; no longer TP7.TESTPOINT
- net SENSORS_SDA: now also U19.SDA; no longer TP5.TESTPOINT
- net SERIAL_NUM: no longer TP13.TESTPOINT
- net TDR_L_DETECT: now also ASSY1.B3
- net TDR_L_TRIGGER: now also ASSY1.B1
- net TDR_N_DETECT: now also ASSY1.B2
- net TDR_N_TRIGGER: now also ASSY1.C1
- net VCC: now also D29.VDD, U19.AD0, U19.AD1, U19.AD2, U19.V+; no longer TP4.TESTPOINT
- net WDI: no longer TP25.TESTPOINT
Other:
- note added: "These resistors *should* give the LEDs the same initial brightness. It accounts for their differing voltage drops and their differing mCD to current ratios. Outputs should be about 12mCd"
- note added: "This driver has integrated brightness control. It's pin compatible with the cheaper PCA9534 (without brightness control). We need it because we are short on pins and still want to drive an LED when we are asleep."
- moved on the sheet: C12, J1, R10, R11, R12, R20, R21, U12

Commit message: make significant layout progress
Parts:
- added C36: 0.1uF, passives:CAPACITOR0402_CAP
- added C37: 1uF, passives:CAPACITOR0402_CAP
- U17, U18, U21, U22: value SN74LVC1G86DBVR -> SN74LVC1G86DRLRDRL5-L; device SN74LVC:SN74LVC1G86DBVR -> SN74LVC1G86:SN74LVC1G86DRLRDRL5-L
Connections:
- new net BOOT0: R37.2, U10.PH3/BOOT0
- net !RST: no longer R37.2, U10.PH3/BOOT0
- net AC_COPROC_VCC: now also C36.1, C37.1
- net GND: now also C36.2, C37.2
Other:
- moved on the sheet: C19, C20, C21, C22, C23
