File: hardware/plugwatch_G/board/plugwatch.sch (EAGLE design)
At the start: 123 parts, among them J1 DM3AT-SF-PEJM5, J2 TC2030-JLINK-L, Q1 MOSFET-NCHANNELSMD, Q2 NX3008PBK, U1 AB1815-T3, U10 MAX7315ATET, U11 REF2030AIDDCR, U12 SIP32510, U13 SIP32510, U14 SIP32510, U19 STM32L432KC, U2 ADA4096-4ACPZ-R7, U20 TCA9406DCUR, U21 TPS79330DBVR, U3 BGA725L6-ALT, U4 DS2401P+, U5 SAFFB1G56KB0F0A, U6 IRM-03-5V, U7 LIS2DH12, U8 MAX-M8, U9 MAX67XXMAX6749MAX67XX, X1 ABS05-32.768KHZ-T, X2 ABS07-32.768KHZ-7-T

Commit message: renaming and a few layout fixes
Parts:
- removed C30: 4.7uF, passives:CAPACITOR0402_CAP
- removed C31, C32: 10uF, passives:CAPACITOR0402_CAP
- removed C33, C34: 100uF, passives:CAPACITOR1210_CAP
- removed C35: 2000uF, rcl:CPOL-USE5-13
- removed R45: 953k, passives:RESISTOR0805_RES
- removed R46, R47, R48: 1M, passives:RESISTOR0402_RES
- added C12, C13: 0.1uF, passives:CAPACITOR0402_CAP
- added C4, C5, C6, C7: 10nF, passives:CAPACITOR0402_CAP
- added R35, R36: 953k, passives:RESISTOR0805_RES
- added R4: 475, passives:RESISTOR0402_RES
- added R5: 750, passives:RESISTOR0402_RES
- C10, C11, C8, C9: value 10nF -> 0.1uF; DESCRIPTION CAP CER 10000PF 16V X7R 0402 -> CAP CER 0.1UF 10V X5R 0402; DIGIKEY 490-1313-1-ND -> 311-1336-1-ND; MANUFACTURER Murata Electronics North America -> Yageo; MPN GRM155R71C103KA01D -> CC0402KRX5R6BB104
- C17: value 0.1uF -> 0.82uF; DESCRIPTION CAP CER 0.1UF 10V X5R 0402 -> CAP CER 0.82UF 10V X5R 0402; DIGIKEY 311-1336-1-ND -> 311-3789-1-ND; MPN CC0402KRX5R6BB104 -> CC0402KRX5R6BB824
- C18, C19, C20, C21: value 0.1uF -> 1uF; DESCRIPTION CAP CER 0.1UF 10V X5R 0402 -> CAP CER 1UF 10V X7S 0402; DIGIKEY 311-1336-1-ND -> 490-13409-1-ND; MANUFACTURER Yageo -> Murata Electronics North America; MPN CC0402KRX5R6BB104 -> GCM155C71A105KE38D
- C22: value 0.1uF -> 2.2uF; DESCRIPTION CAP CER 0.1UF 10V X5R 0402 -> (none); DIGIKEY 311-1336-1-ND -> 490-12696-1-ND; MANUFACTURER Yageo -> Murata Electronics North America; MPN CC0402KRX5R6BB104 -> GRM155C70J225KE11D
- C23: value 0.82uF -> 4.7uF; DESCRIPTION CAP CER 0.82UF 10V X5R 0402 -> CAP CER 4.7UF 6.3V X5R 0402; DIGIKEY 311-3789-1-ND -> 445-5947-1-ND; MANUFACTURER Yageo -> TDK Corporation; MPN CC0402KRX5R6BB824 -> C1005X5R0J475K050BC
- C24: value 1uF -> 4.7uF; DESCRIPTION CAP CER 1UF 10V X7S 0402 -> CAP CER 4.7UF 6.3V X5R 0402; DIGIKEY 490-13409-1-ND -> 445-5947-1-ND; MANUFACTURER Murata Electronics North America -> TDK Corporation; MPN GCM155C71A105KE38D -> C1005X5R0J475K050BC
- C25, C26: value 1uF -> 10uF; DESCRIPTION CAP CER 1UF 10V X7S 0402 -> CAP CER 10UF 6.3V X5R 0402; DIGIKEY 490-13409-1-ND -> 490-13211-1-ND; MPN GCM155C71A105KE38D -> GRJ155R60J106ME11D
- C27: value 1uF -> 100uF; device passives:CAPACITOR0402_CAP -> passives:CAPACITOR1210_CAP; DESCRIPTION CAP CER 1UF 10V X7S 0402 -> CAP CER 100UF 6.3V X7S 1210; DIGIKEY 490-13409-1-ND -> 490-10530-1-ND; MPN GCM155C71A105KE38D -> GRM32EC70J107ME15L
- C28: value 2.2uF -> 100uF; device passives:CAPACITOR0402_CAP -> passives:CAPACITOR1210_CAP; DESCRIPTION (none) -> CAP CER 100UF 6.3V X7S 1210; DIGIKEY 490-12696-1-ND -> 490-10530-1-ND; MPN GRM155C70J225KE11D -> GRM32EC70J107ME15L
- C29: value 4.7uF -> 2000uF; device passives:CAPACITOR0402_CAP -> rcl:CPOL-USE5-13; DESCRIPTION CAP CER 4.7UF 6.3V X5R 0402 -> CAP ALUM 2000UF 20% 6.3V T/H; DIGIKEY 445-5947-1-ND -> P122284TB-ND; MANUFACTURER TDK Corporation -> Panasonic Electronic Components; MPN C1005X5R0J475K050BC -> EEU-FS0J202B
- R10, R11: value 1.69k -> 3.74k; DESCRIPTION RES SMD 1.69K OHM 1% 1/16W 0402 -> RES SMD 3.74KOHM 0.1% 1/16W 0402; DIGIKEY YAG3044CT-ND -> P3.74KDCCT-ND; MANUFACTURER Yageo -> Panasonic Electronic Components; MPN RC0402FR-071K69L -> ERA-2AEB3741X
- R12: value 3.74k -> 5.1k; DESCRIPTION RES SMD 3.74KOHM 0.1% 1/16W 0402 -> RES SMD 5.1K OHM 1% 1/10W 0402; DIGIKEY P3.74KDCCT-ND -> P5.10KLCT-ND; MPN ERA-2AEB3741X -> ERJ-2RKF5101X
- R13: value 3.74k -> 10k; DESCRIPTION RES SMD 3.74KOHM 0.1% 1/16W 0402 -> RES SMD 10K OHM 1% 1/16W 0402; DIGIKEY P3.74KDCCT-ND -> RMCF0402FT10K0CT-ND; MANUFACTURER Panasonic Electronic Components -> Stackpole Electronics Inc.; MPN ERA-2AEB3741X -> RMCF0402FT10K0
- R14: value 5.1k -> 10k; DESCRIPTION RES SMD 5.1K OHM 1% 1/10W 0402 -> RES SMD 10K OHM 1% 1/16W 0402; DIGIKEY P5.10KLCT-ND -> RMCF0402FT10K0CT-ND; MANUFACTURER Panasonic Electronic Components -> Stackpole Electronics Inc.; MPN ERJ-2RKF5101X -> RMCF0402FT10K0
- R23: DESCRIPTION RES SMD 10K OHM 1% 1/16W 0402 -> RES SMD 10K OHM 1% 1/16W 0402; DIGIKEY RMCF0402FT10K0CT-ND -> RMCF0402FT10K0CT-ND; MANUFACTURER Stackpole Electronics Inc. -> Stackpole Electronics Inc.; MPN RMCF0402FT10K0 -> RMCF0402FT10K0
- R24: value 10k -> 34k; DESCRIPTION RES SMD 10K OHM 1% 1/16W 0402 -> RES SMD 34K OHM 1% 1/10W 0402; DIGIKEY RMCF0402FT10K0CT-ND -> P34.0KLCT-ND; MANUFACTURER Stackpole Electronics Inc. -> Panasonic Electronic Components; MPN RMCF0402FT10K0 -> ERJ-2RKF3402X
- R25: value 10k -> 66.5k; DESCRIPTION RES SMD 10K OHM 1% 1/16W 0402 -> RES SMD 66.5K OHM 1% 1/16W 0402; DIGIKEY RMCF0402FT10K0CT-ND -> YAG3209CT-ND; MANUFACTURER Stackpole Electronics Inc. -> Yageo; MPN RMCF0402FT10K0 -> RC0402FR-0766K5L
- R26: value 34k -> 100k; DESCRIPTION RES SMD 34K OHM 1% 1/10W 0402 -> RES SMD 100K OHM 1% 1/16W 0402; DIGIKEY P34.0KLCT-ND -> 311-100KLRCT-ND; MANUFACTURER Panasonic Electronic Components -> Yageo; MPN ERJ-2RKF3402X -> RC0402FR-07100KL
- R27: value 66.5k -> 100k; DESCRIPTION RES SMD 66.5K OHM 1% 1/16W 0402 -> RES SMD 100K OHM 1% 1/16W 0402; DIGIKEY YAG3209CT-ND -> 311-100KLRCT-ND; MPN RC0402FR-0766K5L -> RC0402FR-07100KL
- R33: value 100k -> 825k; DESCRIPTION RES SMD 100K OHM 1% 1/16W 0402 -> RES SMD 825K OHM 1% 1/10W 0402; DIGIKEY 311-100KLRCT-ND -> P825KLCT-ND; MANUFACTURER Yageo -> Panasonic Electronic Components; MPN RC0402FR-07100KL -> ERJ-2RKF8253X
- R34: value 100k -> 953k; device passives:RESISTOR0402_RES -> passives:RESISTOR0805_RES; DESCRIPTION RES SMD 100K OHM 1% 1/16W 0402 -> RES SMD 953K OHM 0.1% 1/8W 0805; DIGIKEY 311-100KLRCT-ND -> P953KDACT-ND; MANUFACTURER Yageo -> Panasonic Electronic Components; MPN RC0402FR-07100KL -> ERA-6AEB9533V
- R37: value 825k -> 953k; device passives:RESISTOR0402_RES -> passives:RESISTOR0805_RES; DESCRIPTION RES SMD 825K OHM 1% 1/10W 0402 -> RES SMD 953K OHM 0.1% 1/8W 0805; DIGIKEY P825KLCT-ND -> P953KDACT-ND; MPN ERJ-2RKF8253X -> ERA-6AEB9533V
- R42, R43, R44: value 953k -> 1M; device passives:RESISTOR0805_RES -> passives:RESISTOR0402_RES; DESCRIPTION RES SMD 953K OHM 0.1% 1/8W 0805 -> RES 1M OHM 1% 1/16W 0402; DIGIKEY P953KDACT-ND -> RMCF0402FT1M00CT-ND; MANUFACTURER Panasonic Electronic Components -> Stackpole Electronics Inc; MPN ERA-6AEB9533V -> RMCF0402FT1M00
- R6: value 475 -> 1.00k; DESCRIPTION RES 475 OHM 1% 1/16W 0402 -> RES SMD 1K OHM 0.1% 1/16W 0402; DIGIKEY RMCF0402FT475RCT-ND -> YAG2306CT-ND; MANUFACTURER Stackpole Electronics Inc -> Yageo; MPN RMCF0402FT475R -> RT0402BRE071KL
- R7: value 750 -> 1.00k; DESCRIPTION RES SMD 750 OHM 1% 1/10W 0402 -> RES SMD 1K OHM 0.1% 1/16W 0402; DIGIKEY P750LCT-ND -> YAG2306CT-ND; MANUFACTURER Panasonic Electronic Components -> Yageo; MPN ERJ-2RKF7500X -> RT0402BRE071KL
- R8, R9: value 1.00k -> 1.69k; DESCRIPTION RES SMD 1K OHM 0.1% 1/16W 0402 -> RES SMD 1.69K OHM 1% 1/16W 0402; DIGIKEY YAG2306CT-ND -> YAG3044CT-ND; MPN RT0402BRE071KL -> RC0402FR-071K69L
- renumbered U19 to U15, U20 to U16, U21 to U17
Connections:
- net !EXTERNAL_RST: now also R21.2; no longer R23.2
- net !RTC_CS: now also R20.2; no longer R24.2
- net !RTC_INT1: now also R19.2; no longer R21.2
- net !RTC_INT2: now also R32.2; no longer R34.2
- net !SD_CS: now also R15.1; no longer R17.1
- net !SD_DETECT: now also R26.1; no longer R28.1
- net 5V: now also C27.1, C28.1, C29.+, R24.1, R29.1, R43.1; no longer C33.1, C34.1, C35.+, R26.1, R31.1, R47.1
- net AC_COPROC_VCC: now also C15.1, C16.1, C20.1, C24.1; no longer C22.1, C26.1, C27.1, C30.1
- net AC_L_800V_DETECT: now also C6.1; no longer C10.1
- net AC_L_HV_OUT: now also R6.2; no longer R8.2
- net AC_L_LV_OUT: now also R10.2; no longer R12.2
- net AC_L_SENSE: now also R34.1, R39.2; no longer R38.1, R43.2
- net AC_N: now also R36.1, R40.2; no longer R40.1, R44.2
- net AC_N_800V_DETECT: now also C7.1; no longer C11.1
- net AC_N_HV_OUT: now also R7.2; no longer R9.2
- net AC_N_LV_OUT: now also R11.1; no longer R13.1
- net AC_SENSE_PWR_EN: now also R31.2; no longer R33.2
- net BOOT0: now also R23.2; no longer R25.2
- net GND: now also C12.2, C13.2, C14.2, C26.1, C29.-, C4.1, C5.1, C6.2, C7.2, C9.2, R18.2, R23.1, R25.2, R27.1, R28.1, R30.2, R31.1, R35.1, R37.1, R38.2, R41.2, R44.2, R9.1; no longer C14.1, C26.2, C29.2, C30.2, C31.2, C32.1, C33.2, C34.2, C35.-, C9.1, R11.1, R20.2, R25.1, R27.2, R29.1, R30.1, R32.2, R33.1, R39.1, R41.1, R45.2, R46.2, R48.2
- net GPS_PWR_EN: now also R28.2; no longer R30.2
- net GPS_VCC: now also C26.2, C5.2, C8.2; no longer C14.2, C32.2, C9.2
- net N$1: now also R9.2; no longer R11.2
- net N$10: now also R24.2, R25.1; no longer R26.2, R27.1
- net N$18: now also C23.1, R14.2, R15.2, R26.2; no longer C29.1, R17.2, R18.2, R28.2
- net N$23: now also R21.1, R33.1; no longer R23.1, R37.1
- net N$25: now also R29.2, R30.1; no longer R31.2, R32.1
- net N$26: now also R4.1; no longer R6.1
- net N$3: now also R11.2, R36.2, R37.2; no longer R13.2, R40.2, R41.2
- net N$31: now also R33.2, R42.1, R43.2; no longer R37.2, R46.1, R47.2
- net N$36: now also C17.1; no longer C23.1
- net N$39: now also C22.1; no longer C28.1
- net N$4: now also R10.1, R34.2, R35.2; no longer R12.1, R38.2, R39.2
- net N$42: now also R5.1; no longer R7.1
- net N$49: now also R8.1; no longer R10.1
- net N$5: now also R22.1; no longer R24.1
- net N$50: now also R8.2; no longer R10.2
- net N$51: now also R5.2; no longer R7.2
- net N$52: now also R4.2; no longer R6.2
- net N$6: now also R38.1, R39.1, R6.1; no longer R42.1, R43.1, R8.1
- net N$8: now also R40.1, R41.1, R7.1; no longer R44.1, R45.1, R9.1
- net PARTICLE_RST: now also R44.1; no longer R48.1
- net REF_1V5: now also C10.1, C11.1, C12.1, C13.1; no longer C16.1, C17.1, C18.1, C19.1
- net REF_3V: now also C14.1, C19.1; no longer C20.1, C25.1
- net SD_ENABLE: now also R27.2; no longer R29.2
- net SD_MISO: now also R16.1; no longer R18.1
- net SD_MOSI: now also R14.1; no longer R16.1
- net SENSORS_SCL: now also R17.1; no longer R19.1
- net SENSORS_SDA: now also R13.1; no longer R15.1
- net SERIAL_NUM: now also R12.2; no longer R14.2
- net VCC: now also C18.1, C25.1, C9.1, R12.1, R13.2, R17.2, R19.1, R20.1, R32.1; no longer C15.1, C24.1, C31.1, R14.1, R15.2, R19.2, R21.1, R22.1, R34.1
- net VCC_RF: now also C4.2; no longer C8.2
- net WDI: now also R18.1; no longer R20.1
