File: hardware/plugwatch_H/board/plugwatch.brd (EAGLE design)
At the start: 55.7 x 95.2 mm, 123 parts, among them J1 DM3AT-SF-PEJM5, J2 TC2030-JLINK-L, Q1 MOSFET-NCHANNELSMD, Q2 NX3008PBK, U1 AB1815-T3, U10 MAX7315ATET, U11 REF2030AIDDCR, U12 SIP32510, U13 SIP32510, U14 SIP32510, U15 STM32L432KC, U16 TCA9406DCUR, U17 TPS79330DBVR, U2 ADA4096-4ACPZ-R7, U3 BGA725L6-ALT, U4 DS2401P+, U5 SAFFB1G56KB0F0A, U6 IRM-03-5V, U7 LIS2DH12, U8 MAX-M8, U9 MAX67XXMAX6749MAX67XX, X1 ABS05-32.768KHZ-T, X2 ABS07-32.768KHZ-7-T

Commit message: update board to fix small issues. BOM should be the same
Parts:
- moved C4 0.51 mm to (44.3, 47.6)
- moved R23 0.51 mm to (6.60, 53.8)
Connections:
- new net VOLTAGE_COPROC_RX: ASSY1.C1, U15.30
- new net VOLTAGE_COPROC_TX: ASSY1.C0, U15.29
- net AC_N_800V_DETECT: now also ASSY1.A1, U15.28; no longer ASSY1.C1, U15.29
- net AC_N_HV_OUT: now also U15.10; no longer U15.8
- net GPS_PWR_EN: now also ASSY1.B2; no longer ASSY1.C0
Routing:
- net AC_N_800V_DETECT: track 70.1 -> 110.6 mm
- net GPS_PWR_EN: track 41.6 -> 60.7 mm
- net VOLTAGE_COPROC_TX: track 0.00 -> 17.6 mm, vias 0 -> 1
- net VOLTAGE_COPROC_RX: track 0.00 -> 16.1 mm, vias 0 -> 1
- net VCC_RF: track 12.8 -> 13.9 mm
- net AC_L_LV_OUT: track 72.6 -> 71.9 mm
Other:
- board text added: "PowerWatch Josh Adkins Noah Klugman Rev H, 11/19"
- board text removed: "PowerWatch Josh Adkins Noah Klugman Rev E, 10/19"
