File: hardware/plugwatch_H/board/plugwatch.sch (EAGLE design)
At the start: 123 parts, among them J1 DM3AT-SF-PEJM5, J2 TC2030-JLINK-L, Q1 MOSFET-NCHANNELSMD, Q2 NX3008PBK, U1 AB1815-T3, U10 MAX7315ATET, U11 REF2030AIDDCR, U12 SIP32510, U13 SIP32510, U14 SIP32510, U15 STM32L432KC, U16 TCA9406DCUR, U17 TPS79330DBVR, U2 ADA4096-4ACPZ-R7, U3 BGA725L6-ALT, U4 DS2401P+, U5 SAFFB1G56KB0F0A, U6 IRM-03-5V, U7 LIS2DH12, U8 MAX-M8, U9 MAX67XXMAX6749MAX67XX, X1 ABS05-32.768KHZ-T, X2 ABS07-32.768KHZ-7-T

Commit message: update board to fix small issues. BOM should be the same
Connections:
- new net VOLTAGE_COPROC_RX: ASSY1.C1, U15.PB7
- new net VOLTAGE_COPROC_TX: ASSY1.C0, U15.PB6
- net AC_N_800V_DETECT: now also ASSY1.A1, U15.PB5; no longer ASSY1.C1, U15.PB6
- net AC_N_HV_OUT: now also U15.PA4; no longer U15.PA2
- net GPS_PWR_EN: now also ASSY1.B2; no longer ASSY1.C0
Other:
- note added: "According to the datasheet these pins are 5.5V tolerant. Turn off when not debugging."
Changed lines of the file:
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@@
 <setting verticaltext="up"/>
 </settings>
-<grid distance="0.1" unitdist="inch" unit="inch" style="lines" multiple="1" display="no" altdistance="0.01" altunitdist="inch" altunit="inch"/>
+<grid distance="0.05" unitdist="inch" unit="inch" style="lines" multiple="1" display="no" altdistance="0.01" altunitdist="inch" altunit="inch"/>
 <layers>
 <layer number="1" name="Top" color="4" fill="1" visible="no" active="no"/>
@@
 <text x="25.4" y="157.48" size="1.27" layer="98">REGULATE 3V3 to 3V so that VDDA
 can be powered by the reference.</text>
+<text x="54.61" y="60.96" size="0.762" layer="98">According to the datasheet
+these pins are 5.5V tolerant.
+Turn off when not debugging.</text>
 </plain>
 <instances>
@@
 <net name="AC_N_800V_DETECT" class="0">
 <segment>
-<pinref part="U15" gate="G$1" pin="PB6"/>
-<wire x1="81.28" y1="71.12" x2="73.66" y2="71.12" width="0.1524" layer="91"/>
-<label x="73.66" y="71.12" size="1.27" layer="95" rot="R180" xref="yes"/>
+<pinref part="U15" gate="G$1" pin="PB5"/>
+<wire x1="81.28" y1="73.66" x2="73.66" y2="73.66" width="0.1524" layer="91"/>
+<label x="73.66" y="73.66" size="1.27" layer="95" rot="R180" xref="yes"/>
 </segment>
 </net>
@@
 <net name="AC_N_HV_OUT" class="0">
 <segment>
-<pinref part="U15" gate="G$1" pin="PA2"/>
-<wire x1="127" y1="91.44" x2="132.08" y2="91.44" width="0.1524" layer="91"/>
-<label x="132.08" y="91.44" size="1.27" layer="95" xref="yes"/>
+<pinref part="U15" gate="G$1" pin="PA4"/>
+<wire x1="127" y1="86.36" x2="132.08" y2="86.36" width="0.1524" layer="91"/>
+<label x="132.08" y="86.36" size="1.27" layer="95" xref="yes"/>
 </segment>
 </net>
@@
 </segment>
 </net>
+<net name="VOLTAGE_COPROC_TX" class="0">
+<segment>
+<pinref part="U15" gate="G$1" pin="PB6"/>
+<wire x1="81.28" y1="71.12" x2="73.66" y2="71.12" width="0.1524" layer="91"/>
+<label x="73.66" y="71.12" size="1.27" layer="95" rot="R180" xref="yes"/>
+</segment>
+</net>
+<net name="VOLTAGE_COPROC_RX" class="0">
+<segment>
+<pinref part="U15" gate="G$1" pin="PB7"/>
+<wire x1="81.28" y1="68.58" x2="73.66" y2="68.58" width="0.1524" layer="91"/>
+<label x="73.66" y="68.58" size="1.27" layer="95" rot="R180" xref="yes"/>
+</segment>
+</net>
 </nets>
 </sheet>
@@
 <net name="GPS_PWR_EN" class="0">
 <segment>
-<pinref part="ASSY1" gate="A1" pin="C0"/>
-<wire x1="100.33" y1="102.87" x2="102.87" y2="102.87" width="0.1524" layer="91"/>
-<label x="102.87" y="102.87" size="1.27" layer="95" xref="yes"/>
+<pinref part="ASSY1" gate="A1" pin="B2"/>
+<wire x1="77.47" y1="107.95" x2="74.93" y2="107.95" width="0.1524" layer="91"/>
+<label x="74.93" y="107.95" size="1.27" layer="95" rot="R180" xref="yes"/>
 </segment>
 </net>
@@
 <net name="AC_N_800V_DETECT" class="0">
 <segment>
-<pinref part="ASSY1" gate="A1" pin="C1"/>
-<wire x1="100.33" y1="105.41" x2="102.87" y2="105.41" width="0.1524" layer="91"/>
-<label x="102.87" y="105.41" size="1.27" layer="95" xref="yes"/>
+<pinref part="ASSY1" gate="A1" pin="A1"/>
+<wire x1="77.47" y1="120.65" x2="74.93" y2="120.65" width="0.1524" layer="91"/>
+<label x="74.93" y="120.65" size="1.27" layer="95" rot="R180" xref="yes"/>
 </segment>
 </net>
@@
 </segment>
 </net>
+<net name="VOLTAGE_COPROC_TX" class="0">
+<segment>
+<pinref part="ASSY1" gate="A1" pin="C0"/>
+<wire x1="100.33" y1="102.87" x2="102.87" y2="102.87" width="0.1524" layer="91"/>
+<label x="102.87" y="102.87" size="1.27" layer="95" xref="yes"/>
+</segment>
+</net>
+<net name="VOLTAGE_COPROC_RX" class="0">
+<segment>
+<pinref part="ASSY1" gate="A1" pin="C1"/>
+<wire x1="100.33" y1="105.41" x2="102.87" y2="105.41" width="0.1524" layer="91"/>
+<label x="102.87" y="105.41" size="1.27" layer="95" xref="yes"/>
+</segment>
+</net>
